File: EE173/EE173_Lab4/EE173_Lab4.sch (KiCad schematic (older format))
At the start: 21 parts

Commit message: Added labels
Parts:
- U?: value Microstrip -> 50ohm
Other:
- note added: "Power Supply"
- note added: "Signal Generator"
Changed lines of the file:
@@
 P 5650 4450
 F 0 "U?" V 5679 4388 50  0000 L CNN
-F 1 "Microstrip" V 5770 4388 50  0000 L CNN
+F 1 "50ohm" V 5770 4388 50  0000 L CNN
 F 2 "" H 5650 4300 50  0001 C CNN
 F 3 "" H 5650 4300 50  0001 C CNN
@@
 	0    1    1    0
 $EndComp
+Wire Notes Line
+	800  800  800  1900
+Wire Notes Line
+	800  1900 3450 1900
+Wire Notes Line
+	3450 1900 3450 800
+Wire Notes Line
+	3450 800  800  800
+Text Notes 950  950  0    50   ~ 0
+Power Supply
+Wire Notes Line
+	2100 3100 2100 4100
+Wire Notes Line
+	2100 4100 600  4100
+Wire Notes Line
+	600  4100 600  3100
+Wire Notes Line
+	600  3100 2100 3100
+Text Notes 700  3200 0    50   ~ 0
+Signal Generator
 $EndSCHEMATC

Commit message: added stupid mofo gate
yyasss
Parts:
- added U?: 4001, symbol 4xxx:4001
- J? (x2): symbol My_Connector:Conn_Coaxial -> EE173_Lab4-rescue:Conn_Coaxial-My_Connector
- U?: symbol My_Schematics:Microstrip -> EE173_Lab4-rescue:Microstrip-My_Schematics
Changed lines of the file:
@@
 EESchema Schematic File Version 4
+LIBS:EE173_Lab4-cache
 EELAYER 26 0
 EELAYER END
@@
 	5500 4100 5500 4150
 $Comp
-L My_Connector:Conn_Coaxial J?
+L EE173_Lab4-rescue:Conn_Coaxial-My_Connector J?
 U 1 1 5BF5C810
 P 6100 4150
@@
 	5500 4150 5900 4150
 $Comp
-L My_Connector:Conn_Coaxial J?
+L EE173_Lab4-rescue:Conn_Coaxial-My_Connector J?
 U 1 1 5BF5CE7C
 P 6100 4850
@@
 	1800 1350 1800 1450
 $Comp
-L My_Schematics:Microstrip U?
+L EE173_Lab4-rescue:Microstrip-My_Schematics U?
 U 1 1 5BF72232
 P 5650 4450
@@
 Text Notes 700  3200 0    50   ~ 0
 Signal Generator
+$Comp
+L 4xxx:4001 U?
+U 1 1 5BF4D94A
+P 8450 1900
+F 0 "U?" H 8450 2225 50  0000 C CNN
+F 1 "4001" H 8450 2134 50  0000 C CNN
+F 2 "" H 8450 1900 50  0001 C CNN
+F 3 "http://www.intersil.com/content/dam/Intersil/documents/cd40/cd4000bms-01bms-02bms-25bms.pdf" H 8450 1900 50  0001 C CNN
+	1    8450 1900
+	1    0    0    -1
+$EndComp
 $EndSCHEMATC

Commit message: Add stupid cap mofo
Parts:
- added C?: C, symbol Device:C
Other:
- moved on the sheet: U?A
Changed lines of the file:
@@
 EESchema Schematic File Version 4
-LIBS:EE173_Lab4-cache
 EELAYER 26 0
 EELAYER END
@@
 L 4xxx:4001 U?
 U 1 1 5BF4D94A
-P 8450 1900
-F 0 "U?" H 8450 2225 50  0000 C CNN
-F 1 "4001" H 8450 2134 50  0000 C CNN
-F 2 "" H 8450 1900 50  0001 C CNN
-F 3 "http://www.intersil.com/content/dam/Intersil/documents/cd40/cd4000bms-01bms-02bms-25bms.pdf" H 8450 1900 50  0001 C CNN
-	1    8450 1900
-	1    0    0    -1
-$EndComp
+P 9600 3400
+F 0 "U?" H 9600 3725 50  0000 C CNN
+F 1 "4001" H 9600 3634 50  0000 C CNN
+F 2 "" H 9600 3400 50  0001 C CNN
+F 3 "http://www.intersil.com/content/dam/Intersil/documents/cd40/cd4000bms-01bms-02bms-25bms.pdf" H 9600 3400 50  0001 C CNN
+	1    9600 3400
+	1    0    0    -1
+$EndComp
+$Comp
+L Device:C C?
+U 1 1 5BF78CB1
+P 8950 3750
+F 0 "C?" H 9065 3796 50  0000 L CNN
+F 1 "C" H 9065 3705 50  0000 L CNN
+F 2 "" H 8988 3600 50  0001 C CNN
+F 3 "~" H 8950 3750 50  0001 C CNN
+	1    8950 3750
+	1    0    0    -1
+$EndComp

Commit message: inductor bois
boi inductors
Parts:
- added L?: L, symbol Device:L
Changed lines of the file:
@@
 EESchema Schematic File Version 4
+LIBS:EE173_Lab4-cache
 EELAYER 26 0
 EELAYER END
@@
 	1    0    0    -1
 $EndComp
+$Comp
+L Device:L L?
+U 1 1 5BF4DBCE
+P 9800 4250
+F 0 "L?" H 9853 4296 50  0000 L CNN
+F 1 "L" H 9853 4205 50  0000 L CNN
+F 2 "" H 9800 4250 50  0001 C CNN
+F 3 "~" H 9800 4250 50  0001 C CNN
+	1    9800 4250
+	1    0    0    -1
+$EndComp

Commit message: Deleted components that were added as a test. Finished some wiring I had overlooked. Added an alternative pulse generator with NOR gates.
Parts:
- removed C?: C, symbol Device:C
- removed L?: L, symbol Device:L
- removed U?: 4001, symbol 4xxx:4001
- added U? (x4): 74HC02, symbol 74xx:74HC02
Connections:
- wire segments 44 -> 57
Other:
- note added: "Alternate pulse generator"
Changed lines of the file:
@@
 Signal Generator
 $Comp
-L 4xxx:4001 U?
-U 1 1 5BF4D94A
-P 9600 3400
-F 0 "U?" H 9600 3725 50  0000 C CNN
-F 1 "4001" H 9600 3634 50  0000 C CNN
-F 2 "" H 9600 3400 50  0001 C CNN
-F 3 "http://www.intersil.com/content/dam/Intersil/documents/cd40/cd4000bms-01bms-02bms-25bms.pdf" H 9600 3400 50  0001 C CNN
-	1    9600 3400
+L 74xx:74HC02 U?
+U 1 1 5BFA238A
+P 2500 4800
+F 0 "U?" H 2500 5125 50  0000 C CNN
+F 1 "74HC02" H 2500 5034 50  0000 C CNN
+F 2 "" H 2500 4800 50  0001 C CNN
+F 3 "http://www.ti.com/lit/gpn/sn74hc02" H 2500 4800 50  0001 C CNN
+	1    2500 4800
 	1    0    0    -1
 $EndComp
 $Comp
-L Device:C C?
-U 1 1 5BF78CB1
-P 8950 3750
-F 0 "C?" H 9065 3796 50  0000 L CNN
-F 1 "C" H 9065 3705 50  0000 L CNN
-F 2 "" H 8988 3600 50  0001 C CNN
-F 3 "~" H 8950 3750 50  0001 C CNN
-	1    8950 3750
+L 74xx:74HC02 U?
+U 2 1 5BFA240B
+P 3150 5550
+F 0 "U?" H 3150 5875 50  0000 C CNN
+F 1 "74HC02" H 3150 5784 50  0000 C CNN
+F 2 "" H 3150 5550 50  0001 C CNN
+F 3 "http://www.ti.com/lit/gpn/sn74hc02" H 3150 5550 50  0001 C CNN
+	2    3150 5550
 	1    0    0    -1
 $EndComp
 $Comp
-L Device:L L?
-U 1 1 5BF4DBCE
-P 9800 4250
-F 0 "L?" H 9853 4296 50  0000 L CNN
-F 1 "L" H 9853 4205 50  0000 L CNN
-F 2 "" H 9800 4250 50  0001 C CNN
-F 3 "~" H 9800 4250 50  0001 C CNN
-	1    9800 4250
+L 74xx:74HC02 U?
+U 3 1 5BFA2492
+P 3850 4900
+F 0 "U?" H 3850 5225 50  0000 C CNN
+F 1 "74HC02" H 3850 5134 50  0000 C CNN
+F 2 "" H 3850 4900 50  0001 C CNN
+F 3 "http://www.ti.com/lit/gpn/sn74hc02" H 3850 4900 50  0001 C CNN
+	3    3850 4900
 	1    0    0    -1
 $EndComp
+$Comp
+L 74xx:74HC02 U?
+U 4 1 5BFA24FF
+P 4750 4900
+F 0 "U?" H 4750 5225 50  0000 C CNN
+F 1 "74HC02" H 4750 5134 50  0000 C CNN
+F 2 "" H 4750 4900 50  0001 C CNN
+F 3 "http://www.ti.com/lit/gpn/sn74hc02" H 4750 4900 50  0001 C CNN
+	4    4750 4900
+	1    0    0    -1
+$EndComp
+Wire Wire Line
+	2800 4800 2850 4800
+Wire Wire Line
+	2850 4800 2850 5450
+Wire Wire Line
+	3450 5550 3450 5000
+$Comp
+L power:GND #PWR?
+U 1 1 5BFA5B7F
+P 2850 5900
+F 0 "#PWR?" H 2850 5650 50  0001 C CNN
+F 1 "GND" H 2855 5727 50  0000 C CNN
+F 2 "" H 2850 5900 50  0001 C CNN
+F 3 "" H 2850 5900 50  0001 C CNN
+	1    2850 5900
+	1    0    0    -1
+$EndComp
+Wire Wire Line
+	2850 5650 2850 5900
+Wire Wire Line
+	2200 4700 2200 4900
+Wire Wire Line
+	4450 4800 4450 4900
+Wire Wire Line
+	4450 4900 4150 4900
+Connection ~ 4450 4900
+Wire Wire Line
+	4450 4900 4450 5000
+Wire Wire Line
+	1150 3650 1150 3800
+$Comp
+L power:GND #PWR?
+U 1 1 5BFAAF3C
+P 4000 2050
+F 0 "#PWR?" H 4000 1800 50  0001 C CNN
+F 1 "GND" H 4005 1877 50  0000 C CNN
+F 2 "" H 4000 2050 50  0001 C CNN
+F 3 "" H 4000 2050 50  0001 C CNN
+	1    4000 2050
+	1    0    0    -1
+$EndComp
+Wire Wire Line
+	3850 1950 4000 1950
+Wire Wire Line
+	4000 1950 4000 2050
+Wire Notes Line
+	2000 4400 5100 4400
+Wire Notes Line
+	5100 4400 5100 6200
+Wire Notes Line
+	5100 6200 2000 6200
+Wire Notes Line
+	2000 6200 2000 4400
+Text Notes 3950 6000 0    50   ~ 0
+Alternate pulse generator
+Wire Wire Line
+	3450 5000 3550 5000
+Wire Wire Line
+	3550 4800 2850 4800
+Connection ~ 2850 4800
 $EndSCHEMATC

Commit message: Added the jumpers to investigate source reflections. Did not choose values for resistors yet
Parts:
- added JP? (x3): Jumper, symbol Device:Jumper
- added R? (x3): R, symbol Device:R
Connections:
- wire segments 57 -> 67
Other:
- moved on the sheet: J?, R?, U?, U?A, U?B, U?C, U?D
