File: EE173/EE173_Lab4/EE173_Lab4.sch (KiCad schematic (older format))
At the start: 31 parts

Commit message: Added BNC connecter at the beginning. This is where we will connect the two microstrips in parallel for the bifurcated line
Parts:
- added J?: Conn_Coaxial, symbol EE173_Lab4-rescue:Conn_Coaxial-My_Connector
- added JP?: Jumper, symbol Device:Jumper
Connections:
- net GND: now also J?.2 (Ext)
- net at C?.2, J?.1 (Pin_1): now also J?.1 (In)
- net at R?.1, R?.1, R?.1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: now also JP?.2
- net at JP?.1, JP?.1, JP?.1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: now also JP?.1
Other:
- note added: "Alt Connection For Bifurcated Line"
- moved on the sheet: C?, D?, J?, JP?, R?, U?, U?A, U?B, U?C, U?D, U?E

Commit message: The BNC connecter at the beginning was a huge mistake. The Bifurcated lines will be added from the other end (OSC connection in Lab 3). Instead I added a jumper at the source to choose between signal generator source or ground. Cleaned up a bit. Added jumper to short for source termination.
Parts:
- removed J?: Conn_Coaxial, symbol EE173_Lab4-rescue:Conn_Coaxial-My_Connector
- added JP? (x2): Jumper, symbol Device:Jumper
Connections:
- net GND: now also R?.2, JP?.1
- net VCC: now also R?.1
- net at J?.1 (Pin_1): now also JP?.1; no longer C?.2
- new net: C?.2, JP?.2, JP?.2
Other:
- note added: "Alt Connection for Bifurcated line"
- note added: "For Grounded Load Terminating Resistors"
- note removed: "Alt Connection For Bifurcated Line"
- moved on the sheet: J?
Changed lines of the file:
@@
 L Connector:Conn_01x02_Male J?
 U 1 1 5BF34C06
-P 3050 4300
-F 0 "J?" H 3156 4478 50  0000 C CNN
-F 1 "Conn_01x02_Male" H 3156 4387 50  0000 C CNN
-F 2 "" H 3050 4300 50  0001 C CNN
-F 3 "~" H 3050 4300 50  0001 C CNN
-	1    3050 4300
-	1    0    0    -1
-$EndComp
-$Comp
-L power:GND #PWR?
+P 2150 3650
+F 0 "J?" H 2256 3828 50  0000 C CNN
+F 1 "Conn_01x02_Male" H 2256 3737 50  0000 C CNN
+F 2 "" H 2150 3650 50  0001 C CNN
+F 3 "~" H 2150 3650 50  0001 C CNN
+	1    2150 3650
+	1    0    0    -1
+$EndComp
+$Comp
+L power:GND #PWR0101
 U 1 1 5BF34E41
-P 3250 4550
-F 0 "#PWR?" H 3250 4300 50  0001 C CNN
-F 1 "GND" H 3255 4377 50  0000 C CNN
-F 2 "" H 3250 4550 50  0001 C CNN
-F 3 "" H 3250 4550 50  0001 C CNN
-	1    3250 4550
+P 2350 3900
+F 0 "#PWR0101" H 2350 3650 50  0001 C CNN
+F 1 "GND" H 2355 3727 50  0000 C CNN
+F 2 "" H 2350 3900 50  0001 C CNN
+F 3 "" H 2350 3900 50  0001 C CNN
+	1    2350 3900
 	1    0    0    -1
 $EndComp
@@
 	0    1    1    0
 $EndComp
-Wire Wire Line
-	3250 4300 3450 4300
 $Comp
 L Device:R R?
@@
 Connection ~ 3900 4300
 $Comp
-L power:VCC #PWR?
+L power:VCC #PWR0102
 U 1 1 5BF3574A
 P 5000 4950
-F 0 "#PWR?" H 5000 4800 50  0001 C CNN
+F 0 "#PWR0102" H 5000 4800 50  0001 C CNN
 F 1 "VCC" V 5018 5077 50  0000 L CNN
 F 2 "" H 5000 4950 50  0001 C CNN
@@
 	8850 5050 8850 5100
 $Comp
-L power:GND #PWR?
+L power:GND #PWR0103
 U 1 1 5BF5C968
 P 9450 5350
-F 0 "#PWR?" H 9450 5100 50  0001 C CNN
+F 0 "#PWR0103" H 9450 5100 50  0001 C CNN
 F 1 "GND" H 9455 5177 50  0000 C CNN
 F 2 "" H 9450 5350 50  0001 C CNN
@@
 $EndComp
 $Comp
-L power:GND #PWR?
+L power:GND #PWR0104
 U 1 1 5BF5CE83
 P 9450 6050
-F 0 "#PWR?" H 9450 5800 50  0001 C CNN
+F 0 "#PWR0104" H 9450 5800 50  0001 C CNN
 F 1 "GND" H 9455 5877 50  0000 C CNN
 F 2 "" H 9450 6050 50  0001 C CNN
@@
 $EndComp
 $Comp
-L power:GND #PWR?
+L power:GND #PWR0105
 U 1 1 5BF62FC3
 P 5650 3850
-F 0 "#PWR?" H 5650 3600 50  0001 C CNN
+F 0 "#PWR0105" H 5650 3600 50  0001 C CNN
 F 1 "GND" H 5655 3677 50  0000 C CNN
 F 2 "" H 5650 3850 50  0001 C CNN
@@
 $EndComp
 $Comp
-L power:GND #PWR?
+L power:GND #PWR0106
 U 1 1 5BF643B0
 P 3900 2200
-F 0 "#PWR?" H 3900 1950 50  0001 C CNN
+F 0 "#PWR0106" H 3900 1950 50  0001 C CNN
 F 1 "GND" H 3905 2027 50  0000 C CNN
 F 2 "" H 3900 2200 50  0001 C CNN
@@
 $EndComp
 $Comp
-L power:GND #PWR?
+L power:GND #PWR0107
 U 1 1 5BF6476A
 P 6700 2050
-F 0 "#PWR?" H 6700 1800 50  0001 C CNN
+F 0 "#PWR0107" H 6700 1800 50  0001 C CNN
 F 1 "GND" H 6705 1877 50  0000 C CNN
 F 2 "" H 6700 2050 50  0001 C CNN
@@
 $EndComp
 $Comp
-L power:GND #PWR?
+L power:GND #PWR0108
 U 1 1 5BF64B24
 P 4850 2400
-F 0 "#PWR?" H 4850 2150 50  0001 C CNN
+F 0 "#PWR0108" H 4850 2150 50  0001 C CNN
 F 1 "GND" H 4855 2227 50  0000 C CNN
 F 2 "" H 4850 2400 50  0001 C CNN
@@
 $EndComp
 $Comp
-L power:GND #PWR?
+L power:GND #PWR0109
 U 1 1 5BF64EDE
 P 5250 2400
-F 0 "#PWR?" H 5250 2150 50  0001 C CNN
+F 0 "#PWR0109" H 5250 2150 50  0001 C CNN
 F 1 "GND" H 5255 2227 50  0000 C CNN
 F 2 "" H 5250 2400 50  0001 C CNN
@@
 $EndComp
 $Comp
-L power:VCC #PWR?
+L power:VCC #PWR0110
 U 1 1 5BF65AF9
 P 5250 1900
-F 0 "#PWR?" H 5250 1750 50  0001 C CNN
+F 0 "#PWR0110" H 5250 1750 50  0001 C CNN
 F 1 "VCC" H 5267 2073 50  0000 C CNN
 F 2 "" H 5250 1900 50  0001 C CNN
@@
 	4450 2000 4550 2000
 $Comp
-L power:GND #PWR?
+L power:GND #PWR0111
 U 1 1 5BF6AE55
 P 4450 2400
-F 0 "#PWR?" H 4450 2150 50  0001 C CNN
+F 0 "#PWR0111" H 4450 2150 50  0001 C CNN
 F 1 "GND" H 4455 2227 50  0000 C CNN
 F 2 "" H 4450 2400 50  0001 C CNN
@@
 Text Notes 3050 1700 0    50   ~ 0
 Power Supply
-Wire Notes Line
-	4200 3850 4200 4850
-Wire Notes Line
-	4200 4850 2700 4850
-Wire Notes Line
-	2700 4850 2700 3850
-Wire Notes Line
-	2700 3850 4200 3850
-Text Notes 2800 3950 0    50   ~ 0
+Text Notes 1900 3300 0    50   ~ 0
 Signal Generator
 $Comp
@@
 	6100 6300 6100 5750
 $Comp
-L power:GND #PWR?
+L power:GND #PWR0112
 U 1 1 5BFA5B7F
 P 5500 6650
-F 0 "#PWR?" H 5500 6400 50  0001 C CNN
+F 0 "#PWR0112" H 5500 6400 50  0001 C CNN
 F 1 "GND" H 5505 6477 50  0000 C CNN
 F 2 "" H 5500 6650 50  0001 C CNN
@@
 	7100 5650 7100 5750
 Wire Wire Line
-	3250 4400 3250 4550
-$Comp
-L power:GND #PWR?
+	2350 3750 2350 3900
+$Comp
+L power:GND #PWR0113
 U 1 1 5BFAAF3C
 P 6100 2800
-F 0 "#PWR?" H 6100 2550 50  0001 C CNN
+F 0 "#PWR0113" H 6100 2550 50  0001 C CNN
 F 1 "GND" H 6105 2627 50  0000 C CNN
 F 2 "" H 6100 2800 50  0001 C CNN
@@
 	8850 4650 8850 4450
 $Comp
-L EE173_Lab4-rescue:Conn_Coaxial-My_Connector J?
-U 1 1 5BFB3354
-P 3450 5500
-F 0 "J?" V 3350 5750 50  0000 L CNN
-F 1 "Conn_Coaxial" V 3250 5550 50  0000 L CNN
-F 2 "" H 3450 5500 50  0001 C CNN
-F 3 " ~" H 3450 5500 50  0001 C CNN
-	1    3450 5500
-	0    1    1    0
-$EndComp
+L Device:Jumper JP?
+U 1 1 5BFC95F1
+P 3150 4200
+F 0 "JP?" H 3150 4350 50  0000 C CNN
+F 1 "Jumper" H 3150 4450 50  0000 C CNN
+F 2 "" H 3150 4200 50  0001 C CNN
+F 3 "~" H 3150 4200 50  0001 C CNN
+	1    3150 4200
+	1    0    0    -1
+$EndComp
+$Comp
+L Device:Jumper JP?
+U 1 1 5BFCA8E8
+P 3150 4400
+F 0 "JP?" H 3150 4200 50  0000 C CNN
+F 1 "Jumper" H 3150 4300 50  0000 C CNN
+F 2 "" H 3150 4400 50  0001 C CNN
+F 3 "~" H 3150 4400 50  0001 C CNN
+	1    3150 4400
+	1    0    0    -1
+$EndComp
+Wire Wire Line
+	3500 4300 3500 4200
+Wire Wire Line
+	3500 4200 3450 4200
+Wire Wire Line
+	3500 4300 3500 4400
+Wire Wire Line
+	3500 4400 3450 4400
+Connection ~ 3500 4300
+$Comp
+L power:VCC #PWR?
+U 1 1 5BFCFBE7
+P 3900 3750
+F 0 "#PWR?" H 3900 3600 50  0001 C CNN
+F 1 "VCC" V 3918 3877 50  0000 L CNN
+F 2 "" H 3900 3750 50  0001 C CNN
+F 3 "" H 3900 3750 50  0001 C CNN
+	1    3900 3750
+	1    0    0    -1
+$EndComp
+Wire Wire Line
+	3900 3950 3900 3750
 $Comp
 L power:GND #PWR?
-U 1 1 5BFB335B
-P 3250 5750
-F 0 "#PWR?" H 3250 5500 50  0001 C CNN
-F 1 "GND" H 3255 5577 50  0000 C CNN
-F 2 "" H 3250 5750 50  0001 C CNN
-F 3 "" H 3250 5750 50  0001 C CNN
-	1    3250 5750
-	1    0    0    -1
-$EndComp
-Wire Wire Line
-	3250 5750 3250 5500
-Wire Wire Line
-	3450 5300 3450 4300
-Connection ~ 3450 4300
-Wire Wire Line
-	3450 4300 3500 4300
-Text Notes 2800 6050 0    50   ~ 0
-Alt Connection For Bifurcated Line
-Wire Notes Line
-	2700 5150 4200 5150
-Wire Notes Line
-	2700 6100 4200 6100
-Wire Notes Line
-	2700 5150 2700 6100
-Wire Notes Line
-	4200 5150 4200 6100
+U 1 1 5BFD3FF6
+P 3900 4800
+F 0 "#PWR?" H 3900 4550 50  0001 C CNN
+F 1 "GND" H 3905 4627 50  0000 C CNN
+F 2 "" H 3900 4800 50  0001 C CNN
+F 3 "" H 3900 4800 50  0001 C CNN
+	1    3900 4800
+	1    0    0    -1
+$EndComp
+Wire Wire Line
+	3900 4650 3900 4800
+Wire Wire Line
+	2350 3650 2650 3650
+Wire Wire Line
+	2650 3650 2650 4200
+Wire Wire Line
+	2650 4200 2850 4200
+$Comp
+L power:GND #PWR?
+U 1 1 5BFDA245
+P 2250 4650
+F 0 "#PWR?" H 2250 4400 50  0001 C CNN
+F 1 "GND" H 2255 4477 50  0000 C CNN
+F 2 "" H 2250 4650 50  0001 C CNN
+F 3 "" H 2250 4650 50  0001 C CNN
+	1    2250 4650
+	1    0    0    -1
+$EndComp
+Wire Wire Line
+	2250 4650 2250 4400
+Wire Wire Line
+	2250 4400 2850 4400
+Wire Notes Line
+	1750 3200 2750 3200
+Wire Notes Line
+	2750 4300 1750 4300
+Wire Notes Line
+	1750 3200 1750 5100
+Text Notes 1800 4950 0    50   ~ 0
+Alt Connection for Bifurcated line
+Text Notes 1800 5050 0    50   ~ 0
+For Grounded Load Terminating Resistors
+Wire Notes Line
+	2750 4850 3400 4850
+Wire Notes Line
+	3400 4850 3400 5100
+Wire Notes Line
+	1750 5100 3400 5100
+Wire Notes Line
+	2750 3200 2750 4850
 $EndSCHEMATC

Commit message: pushed changes i finna delete
Parts:
- removed U? (x4): 74HC02, symbol 74xx:74HC02
- C1, C2, C3, C4: renamed from C?; footprint (none) -> Capacitor_SMD:C_0805_2012Metric
- D2: renamed from D?; footprint (none) -> LED_SMD:LED_0805_2012Metric
- J1, J2: renamed from J?; footprint (none) -> Connector_Pin:Pin_D0.7mm_L6.5mm_W1.8mm_FlatFork
- J3, J4: renamed from J?; footprint (none) -> Connector_Coaxial:BNC_PanelMountable_Vertical
- JP1, JP2, JP3, JP4, JP5, JP6: renamed from JP?; footprint (none) -> Jumper:SolderJumper-2_P1.3mm_Bridged2Bar_Pad1.0x1.5mm
- R1, R2, R3, R4, R5, R6, R7: renamed from R?; footprint (none) -> Resistor_SMD:R_0805_2012Metric
- gave numbers to parts that had none: 4
Other:
- note removed: "Alternate pulse generator"

Commit message: short to one of the jumpers
Parts:
- removed R4: R, Resistor_SMD:R_0805_2012Metric, symbol Device:R
Connections:
- net GND: now also JP3.1
- net at JP6.2, R5.1, R6.1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: now also JP3.2
- net at JP4.1, JP5.1, JP6.1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: no longer JP3.1
Changed lines of the file:
@@
-$EndComp
-$Comp
-L Device:R R4
-U 1 1 5BFA4BB6
-P 8500 3750
-F 0 "R4" V 8293 3750 50  0000 C CNN
-F 1 "R" V 8384 3750 50  0000 C CNN
-F 2 "Resistor_SMD:R_0805_2012Metric" V 8430 3750 50  0001 C CNN
-F 3 "~" H 8500 3750 50  0001 C CNN
-	1    8500 3750
-	0    1    1    0
 $EndComp
 $Comp
@@
 Connection ~ 7600 4450
 Wire Wire Line
-	7600 4100 7600 3750
-Connection ~ 7600 4100
-Wire Wire Line
-	8200 3750 8350 3750
-Wire Wire Line
 	8200 4100 8350 4100
 Wire Wire Line
@@
 Wire Wire Line
 	8850 4700 8850 4650
-Wire Wire Line
-	8850 3750 8650 3750
 Wire Wire Line
 	8650 4100 8850 4100
@@
 Wire Notes Line
 	2750 3200 2750 4850
+Wire Wire Line
+	8200 3750 8850 3750
+$Comp
+L power:GND #PWR?
+U 1 1 5BFD4519
+P 7450 3850
+F 0 "#PWR?" H 7450 3600 50  0001 C CNN
+F 1 "GND" H 7455 3677 50  0000 C CNN
+F 2 "" H 7450 3850 50  0001 C CNN
+F 3 "" H 7450 3850 50  0001 C CNN
+	1    7450 3850
+	1    0    0    -1
+$EndComp
+Wire Wire Line
+	7600 3750 7450 3750
+Wire Wire Line
+	7450 3750 7450 3850
 $EndSCHEMATC

Commit message: deleted microstrip, completed netlist
Parts:
- removed U3: 50ohm, symbol EE173_Lab4-rescue:Microstrip-My_Schematics
- J3: value Conn_Coaxial -> Test Line; footprint Connector_Coaxial:BNC_PanelMountable_Vertical -> My_Footprints:Vertical_BNC_Connector
- J4: value Conn_Coaxial -> OSC
- U1: footprint (none) -> My_Footprints:HC00
- U2: footprint (none) -> My_Footprints:L7806ABV
Connections:
- net at J3.1 (In), R7.2: now also J4.1 (In)
Changed lines of the file:
@@
 P 9450 5050
 F 0 "J3" H 9549 5026 50  0000 L CNN
-F 1 "Conn_Coaxial" H 9549 4935 50  0000 L CNN
-F 2 "Connector_Coaxial:BNC_PanelMountable_Vertical" H 9450 5050 50  0001 C CNN
+F 1 "Test Line" H 9549 4935 50  0000 L CNN
+F 2 "My_Footprints:Vertical_BNC_Connector" H 9450 5050 50  0001 C CNN
 F 3 " ~" H 9450 5050 50  0001 C CNN
 	1    9450 5050
@@
 $EndComp
 Connection ~ 8850 5050
-Wire Wire Line
-	8850 5050 8850 5100
 $Comp
 L power:GND #PWR014
@@
 P 9450 5750
 F 0 "J4" H 9549 5726 50  0000 L CNN
-F 1 "Conn_Coaxial" H 9549 5635 50  0000 L CNN
+F 1 "OSC" H 9549 5635 50  0000 L CNN
 F 2 "Connector_Coaxial:BNC_PanelMountable_Vertical" H 9450 5750 50  0001 C CNN
 F 3 " ~" H 9450 5750 50  0001 C CNN
@@
 F 0 "U2" H 4850 2242 50  0000 C CNN
 F 1 "L7806" H 4850 2151 50  0000 C CNN
-F 2 "" H 4875 1850 50  0001 L CIN
+F 2 "My_Footprints:L7806ABV" H 4875 1850 50  0001 L CIN
 F 3 "http://www.st.com/content/ccc/resource/technical/document/datasheet/41/4f/b3/b0/12/d4/47/88/CD00000444.pdf/files/CD00000444.pdf/jcr:content/translations/en.CD00000444.pdf" H 4850 1950 50  0001 C CNN
 	1    4850 2000
@@
 F 0 "U1" H 4800 4625 50  0000 C CNN
 F 1 "74HC00" H 4800 4534 50  0000 C CNN
-F 2 "" H 4800 4300 50  0001 C CNN
+F 2 "My_Footprints:HC00" H 4800 4300 50  0001 C CNN
 F 3 "http://www.ti.com/lit/gpn/sn74hc00" H 4800 4300 50  0001 C CNN
 	1    4800 4300
@@
 F 0 "U1" H 7100 4775 50  0000 C CNN
 F 1 "74HC00" H 7100 4684 50  0000 C CNN
-F 2 "" H 7100 4450 50  0001 C CNN
+F 2 "My_Footprints:HC00" H 7100 4450 50  0001 C CNN
 F 3 "http://www.ti.com/lit/gpn/sn74hc00" H 7100 4450 50  0001 C CNN
 	2    7100 4450
@@
 F 0 "U1" H 5500 5175 50  0000 C CNN
 F 1 "74HC00" H 5500 5084 50  0000 C CNN
-F 2 "" H 5500 4850 50  0001 C CNN
+F 2 "My_Footprints:HC00" H 5500 4850 50  0001 C CNN
 F 3 "http://www.ti.com/lit/gpn/sn74hc00" H 5500 4850 50  0001 C CNN
 	3    5500 4850
@@
 F 0 "U1" H 6250 4775 50  0000 C CNN
 F 1 "74HC00" H 6250 4684 50  0000 C CNN
-F 2 "" H 6250 4450 50  0001 C CNN
+F 2 "My_Footprints:HC00" H 6250 4450 50  0001 C CNN
 F 3 "http://www.ti.com/lit/gpn/sn74hc00" H 6250 4450 50  0001 C CNN
 	4    6250 4450
@@
 F 0 "U1" H 5880 3296 50  0000 L CNN
 F 1 "74HC00" H 5880 3205 50  0000 L CNN
-F 2 "" H 5650 3250 50  0001 C CNN
+F 2 "My_Footprints:HC00" H 5650 3250 50  0001 C CNN
 F 3 "http://www.ti.com/lit/gpn/sn74hc00" H 5650 3250 50  0001 C CNN
 	5    5650 3250
@@
 Wire Wire Line
 	3900 2100 3900 2200
-$Comp
-L EE173_Lab4-rescue:Microstrip-My_Schematics U3
-U 1 1 5BF72232
-P 9000 5350
-F 0 "U3" V 9029 5288 50  0000 L CNN
-F 1 "50ohm" V 9120 5288 50  0000 L CNN
-F 2 "" H 9000 5200 50  0001 C CNN
-F 3 "" H 9000 5200 50  0001 C CNN
-	1    9000 5350
-	0    1    1    0
-$EndComp
 Wire Notes Line
 	2900 1550 2900 2650
@@
 	8200 3750 8850 3750
 $Comp
-L power:GND #PWR?
+L power:GND #PWR0101
 U 1 1 5BFD4519
 P 7450 3850
-F 0 "#PWR?" H 7450 3600 50  0001 C CNN
+F 0 "#PWR0101" H 7450 3600 50  0001 C CNN
 F 1 "GND" H 7455 3677 50  0000 C CNN
 F 2 "" H 7450 3850 50  0001 C CNN
@@
 Wire Wire Line
 	7450 3750 7450 3850
+Wire Wire Line
+	8850 5050 8850 5750
 $EndSCHEMATC
