File: EE173/Luis/EE173_Lab4.sch (KiCad schematic (older format))
At the start: 24 parts, among them J1 Conn_01x02_Male, J2 Conn_01x02_Male, J3 Test Line, J4 OSC, U1 74HC00, U2 L7806

Commit message: Redid BNC horizontal connector. Updated netlist.
Parts:
- D2: footprint LED_SMD:LED_0805_2012Metric -> LED_THT:LED_D5.0mm
- J1, J2: footprint Connector_Pin:Pin_D0.7mm_L6.5mm_W1.8mm_FlatFork -> My_Footprints:header_2_pins
- J4: footprint Connector_Coaxial:BNC_PanelMountable_Vertical -> My_Footprints:BNC_Connector
- JP1, JP2, JP3, JP4, JP5, JP6: footprint Jumper:SolderJumper-2_P1.3mm_Bridged2Bar_Pad1.0x1.5mm -> My_Footprints:header_2_pins
Connections:
- net GND: now also JP2.2; no longer JP2.1
- net at J1.1 (Pin_1): now also JP1.2; no longer JP1.1
- new net: C1.2, JP1.1, JP2.1
Other:
- note added: "Microstrip"
- moved on the sheet: JP1, JP2
Changed lines of the file:
@@
 F 0 "J1" H 2256 3828 50  0000 C CNN
 F 1 "Conn_01x02_Male" H 2256 3737 50  0000 C CNN
-F 2 "Connector_Pin:Pin_D0.7mm_L6.5mm_W1.8mm_FlatFork" H 2150 3650 50  0001 C CNN
+F 2 "My_Footprints:header_2_pins" H 2150 3650 50  0001 C CNN
 F 3 "~" H 2150 3650 50  0001 C CNN
 	1    2150 3650
@@
 F 0 "J4" H 9549 5726 50  0000 L CNN
 F 1 "OSC" H 9549 5635 50  0000 L CNN
-F 2 "Connector_Coaxial:BNC_PanelMountable_Vertical" H 9450 5750 50  0001 C CNN
+F 2 "My_Footprints:BNC_Connector" H 9450 5750 50  0001 C CNN
 F 3 " ~" H 9450 5750 50  0001 C CNN
 	1    9450 5750
@@
 F 0 "J2" H 3756 2178 50  0000 C CNN
 F 1 "Conn_01x02_Male" H 3350 2100 50  0000 C CNN
-F 2 "Connector_Pin:Pin_D0.7mm_L6.5mm_W1.8mm_FlatFork" H 3650 2000 50  0001 C CNN
+F 2 "My_Footprints:header_2_pins" H 3650 2000 50  0001 C CNN
 F 3 "~" H 3650 2000 50  0001 C CNN
 	1    3650 2000
@@
 F 0 "D2" H 6392 1745 50  0000 C CNN
 F 1 "LED" H 6392 1836 50  0000 C CNN
-F 2 "LED_SMD:LED_0805_2012Metric" H 6400 2000 50  0001 C CNN
+F 2 "LED_THT:LED_D5.0mm" H 6400 2000 50  0001 C CNN
 F 3 "~" H 6400 2000 50  0001 C CNN
 	1    6400 2000
@@
 F 0 "JP3" H 7900 4014 50  0000 C CNN
 F 1 "Jumper" H 7900 3923 50  0000 C CNN
-F 2 "Jumper:SolderJumper-2_P1.3mm_Bridged2Bar_Pad1.0x1.5mm" H 7900 3750 50  0001 C CNN
+F 2 "My_Footprints:header_2_pins" H 7900 3750 50  0001 C CNN
 F 3 "~" H 7900 3750 50  0001 C CNN
 	1    7900 3750
@@
 F 0 "JP4" H 7900 4364 50  0000 C CNN
 F 1 "Jumper" H 7900 4273 50  0000 C CNN
-F 2 "Jumper:SolderJumper-2_P1.3mm_Bridged2Bar_Pad1.0x1.5mm" H 7900 4100 50  0001 C CNN
+F 2 "My_Footprints:header_2_pins" H 7900 4100 50  0001 C CNN
 F 3 "~" H 7900 4100 50  0001 C CNN
 	1    7900 4100
@@
 F 0 "JP5" H 7900 4714 50  0000 C CNN
 F 1 "Jumper" H 7900 4623 50  0000 C CNN
-F 2 "Jumper:SolderJumper-2_P1.3mm_Bridged2Bar_Pad1.0x1.5mm" H 7900 4450 50  0001 C CNN
+F 2 "My_Footprints:header_2_pins" H 7900 4450 50  0001 C CNN
 F 3 "~" H 7900 4450 50  0001 C CNN
 	1    7900 4450
@@
 F 0 "JP6" H 7900 4450 50  0000 C CNN
 F 1 "Jumper" H 7900 4550 50  0000 C CNN
-F 2 "Jumper:SolderJumper-2_P1.3mm_Bridged2Bar_Pad1.0x1.5mm" H 7900 4650 50  0001 C CNN
+F 2 "My_Footprints:header_2_pins" H 7900 4650 50  0001 C CNN
 F 3 "~" H 7900 4650 50  0001 C CNN
 	1    7900 4650
@@
 U 1 1 5BFC95F1
 P 3150 4200
-F 0 "JP1" H 3150 4350 50  0000 C CNN
-F 1 "Jumper" H 3150 4450 50  0000 C CNN
-F 2 "Jumper:SolderJumper-2_P1.3mm_Bridged2Bar_Pad1.0x1.5mm" H 3150 4200 50  0001 C CNN
+F 0 "JP1" H 3150 4550 50  0000 C CNN
+F 1 "Jumper" H 3150 4600 50  0000 C CNN
+F 2 "My_Footprints:header_2_pins" H 3150 4200 50  0001 C CNN
 F 3 "~" H 3150 4200 50  0001 C CNN
 	1    3150 4200
-	1    0    0    -1
+	-1   0    0    1
 $EndComp
 $Comp
@@
 U 1 1 5BFCA8E8
 P 3150 4400
-F 0 "JP2" H 3150 4200 50  0000 C CNN
-F 1 "Jumper" H 3150 4300 50  0000 C CNN
-F 2 "Jumper:SolderJumper-2_P1.3mm_Bridged2Bar_Pad1.0x1.5mm" H 3150 4400 50  0001 C CNN
+F 0 "JP2" H 3150 4000 50  0000 C CNN
+F 1 "Jumper" H 3150 4050 50  0000 C CNN
+F 2 "My_Footprints:header_2_pins" H 3150 4400 50  0001 C CNN
 F 3 "~" H 3150 4400 50  0001 C CNN
 	1    3150 4400
-	1    0    0    -1
+	-1   0    0    1
 $EndComp
 Wire Wire Line
@@
 Wire Wire Line
 	8850 5050 8850 5750
+Wire Notes Line
+	8750 5150 8950 5150
+Wire Notes Line
+	8950 5150 8950 5650
+Wire Notes Line
+	8950 5650 8750 5650
+Wire Notes Line
+	8750 5650 8750 5150
+Text Notes 8750 5600 1    50   ~ 0
+Microstrip
 $EndSCHEMATC

Commit message: worked on layout
Connections:
- net at JP3.2, JP6.2, R5.1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: now also J3.1 (In)
- net at J4.1 (In), R7.2: no longer J3.1 (In)
Other:
- moved on the sheet: J4, R7
Changed lines of the file:
@@
 L Device:R R7
 U 1 1 5BF35A5D
-P 8850 4850
-F 0 "R7" H 8920 4896 50  0000 L CNN
-F 1 "R" H 8920 4805 50  0000 L CNN
-F 2 "Resistor_SMD:R_0805_2012Metric" V 8780 4850 50  0001 C CNN
-F 3 "~" H 8850 4850 50  0001 C CNN
-	1    8850 4850
-	1    0    0    -1
-$EndComp
-Wire Wire Line
-	8850 5000 8850 5050
+P 8850 5250
+F 0 "R7" H 8920 5296 50  0000 L CNN
+F 1 "R" H 8920 5205 50  0000 L CNN
+F 2 "Resistor_SMD:R_0805_2012Metric" V 8780 5250 50  0001 C CNN
+F 3 "~" H 8850 5250 50  0001 C CNN
+	1    8850 5250
+	1    0    0    -1
+$EndComp
 $Comp
 L EE173_Lab4-rescue:Conn_Coaxial-My_Connector J3
@@
 	1    0    0    -1
 $EndComp
-Connection ~ 8850 5050
 $Comp
 L power:GND #PWR014
@@
 L EE173_Lab4-rescue:Conn_Coaxial-My_Connector J4
 U 1 1 5BF5CE7C
-P 9450 5750
-F 0 "J4" H 9549 5726 50  0000 L CNN
-F 1 "OSC" H 9549 5635 50  0000 L CNN
-F 2 "My_Footprints:BNC_Connector" H 9450 5750 50  0001 C CNN
-F 3 " ~" H 9450 5750 50  0001 C CNN
-	1    9450 5750
+P 9450 6100
+F 0 "J4" H 9549 6076 50  0000 L CNN
+F 1 "OSC" H 9549 5985 50  0000 L CNN
+F 2 "My_Footprints:BNC_Connector" H 9450 6100 50  0001 C CNN
+F 3 " ~" H 9450 6100 50  0001 C CNN
+	1    9450 6100
 	1    0    0    -1
 $EndComp
@@
 L power:GND #PWR015
 U 1 1 5BF5CE83
-P 9450 6050
-F 0 "#PWR015" H 9450 5800 50  0001 C CNN
-F 1 "GND" H 9455 5877 50  0000 C CNN
-F 2 "" H 9450 6050 50  0001 C CNN
-F 3 "" H 9450 6050 50  0001 C CNN
-	1    9450 6050
-	1    0    0    -1
-$EndComp
-Wire Wire Line
-	9450 6050 9450 5950
-Wire Wire Line
-	8850 5750 9250 5750
+P 9450 6400
+F 0 "#PWR015" H 9450 6150 50  0001 C CNN
+F 1 "GND" H 9455 6227 50  0000 C CNN
+F 2 "" H 9450 6400 50  0001 C CNN
+F 3 "" H 9450 6400 50  0001 C CNN
+	1    9450 6400
+	1    0    0    -1
+$EndComp
+Wire Wire Line
+	9450 6400 9450 6300
+Wire Wire Line
+	8850 6100 9250 6100
 $Comp
 L Regulator_Linear:L7806 U2
@@
 	8200 4450 8350 4450
 Wire Wire Line
-	8850 4700 8850 4650
-Wire Wire Line
 	8650 4100 8850 4100
 Connection ~ 8850 4100
@@
 Wire Wire Line
 	7450 3750 7450 3850
-Wire Wire Line
-	8850 5050 8850 5750
-Wire Notes Line
-	8750 5150 8950 5150
-Wire Notes Line
-	8950 5150 8950 5650
-Wire Notes Line
-	8950 5650 8750 5650
-Wire Notes Line
-	8750 5650 8750 5150
-Text Notes 8750 5600 1    50   ~ 0
+Wire Notes Line
+	8750 5450 8950 5450
+Wire Notes Line
+	8950 5450 8950 5950
+Wire Notes Line
+	8950 5950 8750 5950
+Wire Notes Line
+	8750 5950 8750 5450
+Text Notes 8750 5900 1    50   ~ 0
 Microstrip
+Wire Wire Line
+	8850 4650 8850 5050
+Wire Wire Line
+	8850 5100 8850 5050
+Connection ~ 8850 5050
+Wire Wire Line
+	8850 5400 8850 6100
 $EndSCHEMATC

Commit message: Finished layout. Changed VCC to 6V.
Connections:
- net at J1.1 (Pin_1): now also JP1.1; no longer JP1.2
- net at C1.2, JP2.1: now also JP1.2; no longer JP1.1
- net VCC renamed +6V
Other:
- moved on the sheet: J2, JP1
Changed lines of the file:
@@
 Connection ~ 3900 4300
-$Comp
-L power:VCC #PWR08
-U 1 1 5BF3574A
-P 5000 4950
-F 0 "#PWR08" H 5000 4800 50  0001 C CNN
-F 1 "VCC" V 5018 5077 50  0000 L CNN
-F 2 "" H 5000 4950 50  0001 C CNN
-F 3 "" H 5000 4950 50  0001 C CNN
-	1    5000 4950
-	0    -1   -1   0
-$EndComp
 $Comp
 L Device:R R7
@@
 L Connector:Conn_01x02_Male J2
 U 1 1 5BF61605
-P 3650 2000
-F 0 "J2" H 3756 2178 50  0000 C CNN
-F 1 "Conn_01x02_Male" H 3350 2100 50  0000 C CNN
-F 2 "My_Footprints:header_2_pins" H 3650 2000 50  0001 C CNN
-F 3 "~" H 3650 2000 50  0001 C CNN
-	1    3650 2000
-	1    0    0    -1
-$EndComp
-Wire Wire Line
-	3850 2000 3950 2000
+P 3600 2000
+F 0 "J2" H 3706 2178 50  0000 C CNN
+F 1 "Conn_01x02_Male" H 3300 2100 50  0000 C CNN
+F 2 "My_Footprints:header_2_pins" H 3600 2000 50  0001 C CNN
+F 3 "~" H 3600 2000 50  0001 C CNN
+	1    3600 2000
+	1    0    0    -1
+$EndComp
 $Comp
 L 74xx:74HC00 U1
@@
 L power:GND #PWR03
 U 1 1 5BF643B0
-P 3900 2200
-F 0 "#PWR03" H 3900 1950 50  0001 C CNN
-F 1 "GND" H 3905 2027 50  0000 C CNN
-F 2 "" H 3900 2200 50  0001 C CNN
-F 3 "" H 3900 2200 50  0001 C CNN
-	1    3900 2200
+P 3850 2200
+F 0 "#PWR03" H 3850 1950 50  0001 C CNN
+F 1 "GND" H 3855 2027 50  0000 C CNN
+F 2 "" H 3850 2200 50  0001 C CNN
+F 3 "" H 3850 2200 50  0001 C CNN
+	1    3850 2200
 	1    0    0    -1
 $EndComp
@@
 	1    0    0    -1
 $EndComp
-$Comp
-L power:VCC #PWR09
-U 1 1 5BF65AF9
-P 5250 1900
-F 0 "#PWR09" H 5250 1750 50  0001 C CNN
-F 1 "VCC" H 5267 2073 50  0000 C CNN
-F 2 "" H 5250 1900 50  0001 C CNN
-F 3 "" H 5250 1900 50  0001 C CNN
-	1    5250 1900
-	1    0    0    -1
-$EndComp
 Wire Wire Line
 	5150 2000 5250 2000
-Wire Wire Line
-	5250 2000 5250 1900
 Connection ~ 5250 2000
 Wire Wire Line
@@
 	4450 2400 4450 2300
 Wire Wire Line
-	3850 2100 3900 2100
-Wire Wire Line
-	3900 2100 3900 2200
+	3800 2100 3850 2100
+Wire Wire Line
+	3850 2100 3850 2200
 Wire Notes Line
 	2900 1550 2900 2650
@@
 U 1 1 5BFC95F1
 P 3150 4200
-F 0 "JP1" H 3150 4550 50  0000 C CNN
-F 1 "Jumper" H 3150 4600 50  0000 C CNN
+F 0 "JP1" H 3150 4350 50  0000 C CNN
+F 1 "Jumper" H 3150 4450 50  0000 C CNN
 F 2 "My_Footprints:header_2_pins" H 3150 4200 50  0001 C CNN
 F 3 "~" H 3150 4200 50  0001 C CNN
 	1    3150 4200
-	-1   0    0    1
+	1    0    0    -1
 $EndComp
 $Comp
@@
 U 1 1 5BFCA8E8
 P 3150 4400
-F 0 "JP2" H 3150 4000 50  0000 C CNN
-F 1 "Jumper" H 3150 4050 50  0000 C CNN
+F 0 "JP2" H 3200 4650 50  0000 C CNN
+F 1 "Jumper" H 3200 4550 50  0000 C CNN
 F 2 "My_Footprints:header_2_pins" H 3150 4400 50  0001 C CNN
 F 3 "~" H 3150 4400 50  0001 C CNN
@@
 	3500 4400 3450 4400
 Connection ~ 3500 4300
-$Comp
-L power:VCC #PWR04
-U 1 1 5BFCFBE7
-P 3900 3750
-F 0 "#PWR04" H 3900 3600 50  0001 C CNN
-F 1 "VCC" V 3918 3877 50  0000 L CNN
-F 2 "" H 3900 3750 50  0001 C CNN
-F 3 "" H 3900 3750 50  0001 C CNN
-	1    3900 3750
-	1    0    0    -1
-$EndComp
 Wire Wire Line
 	3900 3950 3900 3750
@@
 Wire Wire Line
 	8850 5400 8850 6100
+$Comp
+L power:+6V #PWR?
+U 1 1 5BFF20A8
+P 5250 1900
+F 0 "#PWR?" H 5250 1750 50  0001 C CNN
+F 1 "+6V" H 5265 2073 50  0000 C CNN
+F 2 "" H 5250 1900 50  0001 C CNN
+F 3 "" H 5250 1900 50  0001 C CNN
+	1    5250 1900
+	1    0    0    -1
+$EndComp
+Wire Wire Line
+	5250 1900 5250 2000
+$Comp
+L power:+6V #PWR?
+U 1 1 5BFF4C96
+P 3900 3750
+F 0 "#PWR?" H 3900 3600 50  0001 C CNN
+F 1 "+6V" H 3915 3923 50  0000 C CNN
+F 2 "" H 3900 3750 50  0001 C CNN
+F 3 "" H 3900 3750 50  0001 C CNN
+	1    3900 3750
+	1    0    0    -1
+$EndComp
+$Comp
+L power:+6V #PWR?
+U 1 1 5BFF788D
+P 5000 4950
+F 0 "#PWR?" H 5000 4800 50  0001 C CNN
+F 1 "+6V" V 5015 5078 50  0000 L CNN
+F 2 "" H 5000 4950 50  0001 C CNN
+F 3 "" H 5000 4950 50  0001 C CNN
+	1    5000 4950
+	0    -1   -1   0
+$EndComp
+Wire Wire Line
+	3800 2000 3950 2000
 $EndSCHEMATC

Commit message: Complete layout. Just need to finalize microstrip length
Changed lines of the file:
@@
 L power:GND #PWR07
 U 1 1 5BF64B24
-P 4850 2400
-F 0 "#PWR07" H 4850 2150 50  0001 C CNN
-F 1 "GND" H 4855 2227 50  0000 C CNN
-F 2 "" H 4850 2400 50  0001 C CNN
-F 3 "" H 4850 2400 50  0001 C CNN
-	1    4850 2400
+P 6800 2750
+F 0 "#PWR07" H 6800 2500 50  0001 C CNN
+F 1 "GND" H 6805 2577 50  0000 C CNN
+F 2 "" H 6800 2750 50  0001 C CNN
+F 3 "" H 6800 2750 50  0001 C CNN
+	1    6800 2750
 	1    0    0    -1
 $EndComp
@@
 L power:GND #PWR06
 U 1 1 5BF6AE55
-P 4450 2400
-F 0 "#PWR06" H 4450 2150 50  0001 C CNN
-F 1 "GND" H 4455 2227 50  0000 C CNN
-F 2 "" H 4450 2400 50  0001 C CNN
-F 3 "" H 4450 2400 50  0001 C CNN
-	1    4450 2400
+P 6400 2750
+F 0 "#PWR06" H 6400 2500 50  0001 C CNN
+F 1 "GND" H 6405 2577 50  0000 C CNN
+F 2 "" H 6400 2750 50  0001 C CNN
+F 3 "" H 6400 2750 50  0001 C CNN
+	1    6400 2750
 	1    0    0    -1
 $EndComp
@@
 	8850 5400 8850 6100
 $Comp
-L power:+6V #PWR?
+L power:+6V #PWR0102
 U 1 1 5BFF20A8
 P 5250 1900
-F 0 "#PWR?" H 5250 1750 50  0001 C CNN
+F 0 "#PWR0102" H 5250 1750 50  0001 C CNN
 F 1 "+6V" H 5265 2073 50  0000 C CNN
 F 2 "" H 5250 1900 50  0001 C CNN
@@
 	5250 1900 5250 2000
 $Comp
-L power:+6V #PWR?
+L power:+6V #PWR0103
 U 1 1 5BFF4C96
 P 3900 3750
-F 0 "#PWR?" H 3900 3600 50  0001 C CNN
+F 0 "#PWR0103" H 3900 3600 50  0001 C CNN
 F 1 "+6V" H 3915 3923 50  0000 C CNN
 F 2 "" H 3900 3750 50  0001 C CNN
@@
 $EndComp
 $Comp
-L power:+6V #PWR?
+L power:+6V #PWR0104
 U 1 1 5BFF788D
 P 5000 4950
-F 0 "#PWR?" H 5000 4800 50  0001 C CNN
+F 0 "#PWR0104" H 5000 4800 50  0001 C CNN
 F 1 "+6V" V 5015 5078 50  0000 L CNN
 F 2 "" H 5000 4950 50  0001 C CNN
@@
 Wire Wire Line
 	3800 2000 3950 2000
+$Comp
+L power:GND #PWR?
+U 1 1 5C00230E
+P 4850 2400
+F 0 "#PWR?" H 4850 2150 50  0001 C CNN
+F 1 "GND" H 4855 2227 50  0000 C CNN
+F 2 "" H 4850 2400 50  0001 C CNN
+F 3 "" H 4850 2400 50  0001 C CNN
+	1    4850 2400
+	1    0    0    -1
+$EndComp
+$Comp
+L power:GND #PWR?
+U 1 1 5C003883
+P 4450 2400
+F 0 "#PWR?" H 4450 2150 50  0001 C CNN
+F 1 "GND" H 4455 2227 50  0000 C CNN
+F 2 "" H 4450 2400 50  0001 C CNN
+F 3 "" H 4450 2400 50  0001 C CNN
+	1    4450 2400
+	1    0    0    -1
+$EndComp
 $EndSCHEMATC
