File: EE173/Luis/EE173_Lab4.sch (KiCad schematic (older format))
At the start: 24 parts, among them J1 Conn_01x02_Male, J2 Conn_01x02_Male, J3 Test Line, J4 OSC, U1 74HC00, U2 L7806

Commit message: added new HC00 Footprint under digikey.pretty
Parts:
- J3: footprint My_Footprints:Vertical_BNC_Connector -> My_Footprints:BNC_Connector
- U1: footprint My_Footprints:HC00 -> digikey:SN74HC00DR
Connections:
- net +6V: now also U1.13; no longer U1.10
- net GND: now also JP3.2; no longer JP3.1
- net at C1.1, R1.2, R2.1: now also U1.10, U1.9; no longer U1.1, U1.2
- net at J3.1 (In), JP6.2, R5.1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: now also JP3.1; no longer JP3.2
- net at U1.4, U1.5: now also U1.3; no longer U1.11
- net at U1.8: now also U1.1, U1.12; no longer U1.13
- new net: U1.11, U1.2
Other:
- moved on the sheet: JP3, U1A, U1C, U1D
Changed lines of the file:
@@
 F 0 "J3" H 9549 5026 50  0000 L CNN
 F 1 "Test Line" H 9549 4935 50  0000 L CNN
-F 2 "My_Footprints:Vertical_BNC_Connector" H 9450 5050 50  0001 C CNN
+F 2 "My_Footprints:BNC_Connector" H 9450 5050 50  0001 C CNN
 F 3 " ~" H 9450 5050 50  0001 C CNN
 	1    9450 5050
@@
 L 74xx:74HC00 U1
 U 1 1 5BF5D5E6
-P 4800 4300
-F 0 "U1" H 4800 4625 50  0000 C CNN
-F 1 "74HC00" H 4800 4534 50  0000 C CNN
-F 2 "My_Footprints:HC00" H 4800 4300 50  0001 C CNN
-F 3 "http://www.ti.com/lit/gpn/sn74hc00" H 4800 4300 50  0001 C CNN
-	1    4800 4300
+P 6250 4450
+F 0 "U1" H 6250 4775 50  0000 C CNN
+F 1 "74HC00" H 6250 4684 50  0000 C CNN
+F 2 "digikey:SN74HC00DR" H 6250 4450 50  0001 C CNN
+F 3 "http://www.ti.com/lit/gpn/sn74hc00" H 6250 4450 50  0001 C CNN
+	1    6250 4450
 	1    0    0    -1
 $EndComp
@@
 F 0 "U1" H 7100 4775 50  0000 C CNN
 F 1 "74HC00" H 7100 4684 50  0000 C CNN
-F 2 "My_Footprints:HC00" H 7100 4450 50  0001 C CNN
+F 2 "digikey:SN74HC00DR" H 7100 4450 50  0001 C CNN
 F 3 "http://www.ti.com/lit/gpn/sn74hc00" H 7100 4450 50  0001 C CNN
 	2    7100 4450
@@
 L 74xx:74HC00 U1
 U 3 1 5BF5D77A
+P 4800 4300
+F 0 "U1" H 4800 4625 50  0000 C CNN
+F 1 "74HC00" H 4800 4534 50  0000 C CNN
+F 2 "digikey:SN74HC00DR" H 4800 4300 50  0001 C CNN
+F 3 "http://www.ti.com/lit/gpn/sn74hc00" H 4800 4300 50  0001 C CNN
+	3    4800 4300
+	1    0    0    -1
+$EndComp
+$Comp
+L 74xx:74HC00 U1
+U 4 1 5BF5D7E4
 P 5500 4850
 F 0 "U1" H 5500 5175 50  0000 C CNN
 F 1 "74HC00" H 5500 5084 50  0000 C CNN
-F 2 "My_Footprints:HC00" H 5500 4850 50  0001 C CNN
+F 2 "digikey:SN74HC00DR" H 5500 4850 50  0001 C CNN
 F 3 "http://www.ti.com/lit/gpn/sn74hc00" H 5500 4850 50  0001 C CNN
-	3    5500 4850
-	1    0    0    -1
-$EndComp
-$Comp
-L 74xx:74HC00 U1
-U 4 1 5BF5D7E4
-P 6250 4450
-F 0 "U1" H 6250 4775 50  0000 C CNN
-F 1 "74HC00" H 6250 4684 50  0000 C CNN
-F 2 "My_Footprints:HC00" H 6250 4450 50  0001 C CNN
-F 3 "http://www.ti.com/lit/gpn/sn74hc00" H 6250 4450 50  0001 C CNN
-	4    6250 4450
+	4    5500 4850
 	1    0    0    -1
 $EndComp
@@
 F 0 "U1" H 5880 3296 50  0000 L CNN
 F 1 "74HC00" H 5880 3205 50  0000 L CNN
-F 2 "My_Footprints:HC00" H 5650 3250 50  0001 C CNN
+F 2 "digikey:SN74HC00DR" H 5650 3250 50  0001 C CNN
 F 3 "http://www.ti.com/lit/gpn/sn74hc00" H 5650 3250 50  0001 C CNN
 	5    5650 3250
@@
 U 1 1 5BFA2C68
 P 7900 3750
-F 0 "JP3" H 7900 4014 50  0000 C CNN
-F 1 "Jumper" H 7900 3923 50  0000 C CNN
+F 0 "JP3" H 7900 3650 50  0000 C CNN
+F 1 "Jumper" H 7900 3550 50  0000 C CNN
 F 2 "My_Footprints:header_2_pins" H 7900 3750 50  0001 C CNN
 F 3 "~" H 7900 3750 50  0001 C CNN
 	1    7900 3750
-	1    0    0    -1
+	-1   0    0    1
 $EndComp
 $Comp
@@
 U 1 1 5BFA2CF7
 P 7900 4100
-F 0 "JP4" H 7900 4364 50  0000 C CNN
+F 0 "JP4" H 7900 4150 50  0000 C CNN
 F 1 "Jumper" H 7900 4273 50  0000 C CNN
 F 2 "My_Footprints:header_2_pins" H 7900 4100 50  0001 C CNN
