File: EE173/Luis/EE173_Lab4.kicad_pcb (KiCad board)
At the start: 2 copper layers, 26 parts, among them J1 Conn_01x02_Male, J2 Conn_01x02_Male, J3 Conn_Coaxial, J4 Conn_Coaxial, U1 74HC00, U2 L7806, U4 50ohm

Commit message: Redid BNC horizontal connector. Updated netlist.
Parts:
- removed R4: R, Resistor_SMD:R_0805_2012Metric
- removed U4: 50ohm, My_Footprints:MicroStrip
- J1, J2: footprint My_Footprints:Two_Pos_Jumper -> Connector_Pin:Pin_D0.7mm_L6.5mm_W1.8mm_FlatFork
- J3: value Conn_Coaxial -> Test Line; footprint My_Footprints:BNC_Connector -> My_Footprints:Vertical_BNC_Connector
- J4: value Conn_Coaxial -> OSC
- JP1, JP2, JP3, JP4, JP5, JP6: footprint My_Footprints:Two_Pos_Jumper -> Jumper:SolderJumper-2_P1.3mm_Bridged2Bar_Pad1.0x1.5mm
- moved D2 67.1 mm to (135.9, 90.2)
- moved JP4 60.4 mm to (227.9, 90.2)
- moved U1 59.0 mm to (134.6, 105.4)
- moved R1 55.2 mm to (155.9, 123.2)
- moved J2 54.7 mm to (125.7, 120.7)
- moved J1 53.8 mm to (125.7, 127.0)
- moved R6 53.8 mm to (161.0, 123.2)
- moved U2 37.3 mm to (146.1, 76.2)
- moved D1 37.3 mm to (156.2, 76.2)
- moved R3 36.7 mm to (155.9, 116.8)
- moved JP2 34.6 mm to (200.0, 87.6)
- moved R7 34.6 mm to (161.6, 116.8)
- moved JP1 32.3 mm to (203.8, 94.0)
- moved R5 31.3 mm to (170.4, 98.7)
- moved JP6 29.7 mm to (210.2, 97.8)
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Connections:
- J4 pad 1: Net-(J4-Pad1) -> Net-(J3-Pad1)
- JP3 pad 1: Net-(JP3-Pad1) -> GND
- JP4 pad 1: Net-(JP3-Pad1) -> Net-(JP4-Pad1)
- JP5 pad 1: Net-(JP3-Pad1) -> Net-(JP4-Pad1)
- JP6 pad 1: Net-(JP3-Pad1) -> Net-(JP4-Pad1)
- JP6 pad 2: Net-(JP6-Pad2) -> Net-(JP3-Pad2)
- R5 pad 1: Net-(JP6-Pad2) -> Net-(JP3-Pad2)
- R6 pad 1: Net-(JP6-Pad2) -> Net-(JP3-Pad2)
- R7 pad 1: Net-(JP6-Pad2) -> Net-(JP3-Pad2)
- U1 pad 6: Net-(JP3-Pad1) -> Net-(JP4-Pad1)

Commit message: worked on layout
Parts:
- J1, J2: footprint Connector_Pin:Pin_D0.7mm_L6.5mm_W1.8mm_FlatFork -> My_Footprints:header_2_pins
- JP1, JP2, JP3, JP4, JP5, JP6: footprint Jumper:SolderJumper-2_P1.3mm_Bridged2Bar_Pad1.0x1.5mm -> My_Footprints:header_2_pins
- moved J2 66.1 mm to (191.8, 124.5)
- moved C3 62.2 mm to (140.0, 104.1)
- moved D2 47.0 mm to (172.7, 61.0)
- moved J1 46.6 mm to (153.4, 89.6)
- moved JP4 44.9 mm to (191.8, 116.8)
- moved R7 43.3 mm to (189.6, 83.8)
- moved JP6 35.6 mm to (191.8, 128.3)
- moved C4 35.6 mm to (128.6, 102.9)
- moved JP5 34.2 mm to (191.8, 120.7)
- moved C2 32.6 mm to (132.4, 104.1)
- moved C1 31.3 mm to (136.2, 104.1)
- moved JP3 25.8 mm to (191.8, 108.0)
- moved R2 24.4 mm to (159.1, 110.5)
- moved J4 22.9 mm to (204.5, 83.8), turned to 90 degrees
- moved JP1 22.6 mm to (191.8, 113.0)
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Connections:
- J4 pad 1: Net-(J3-Pad1) -> Net-(J4-Pad1)
- JP1 pad 1: Net-(J1-Pad1) -> Net-(C1-Pad2)
- JP1 pad 2: Net-(C1-Pad2) -> Net-(J1-Pad1)
- JP2 pad 1: GND -> Net-(C1-Pad2)
- JP2 pad 2: Net-(C1-Pad2) -> GND
- JP3 pad 2: Net-(JP3-Pad2) -> Net-(J3-Pad1)
- JP6 pad 2: Net-(JP3-Pad2) -> Net-(J3-Pad1)
- R5 pad 1: Net-(JP3-Pad2) -> Net-(J3-Pad1)
- R6 pad 1: Net-(JP3-Pad2) -> Net-(J3-Pad1)
- R7 pad 1: Net-(JP3-Pad2) -> Net-(J3-Pad1)
- R7 pad 2: Net-(J3-Pad1) -> Net-(J4-Pad1)
Routing:
- net Net-(J3-Pad1): track 0.00 -> 5.75 mm
- added copper zone on F.Cu, net Net-(J4-Pad1)

Commit message: Finished layout. Changed VCC to 6V.
Parts:
- moved J2 88.2 mm to (150.2, 46.6), turned to 270 degrees
- moved JP1 61.6 mm to (137.3, 84.3), turned to 270 degrees
- moved C2 58.1 mm to (157.9, 51.9)
- moved JP2 56.5 mm to (137.3, 89.3), turned to 270 degrees
- moved R3 50.6 mm to (173.4, 63.2), turned to 180 degrees
- moved C4 48.2 mm to (173.6, 85.6), turned to 180 degrees
- moved C3 47.0 mm to (163.7, 63.5), turned to 90 degrees
- moved D1 41.0 mm to (163.7, 46.6), turned to 180 degrees
- moved R6 32.8 mm to (192.6, 96.6), turned to 180 degrees
- moved JP6 28.8 mm to (185.7, 100.1)
- moved R5 27.1 mm to (192.6, 93.1), turned to 180 degrees
- moved JP5 24.8 mm to (185.7, 96.6)
- moved JP4 24.5 mm to (185.7, 93.1)
- moved R1 21.9 mm to (154.2, 88.7), turned to 270 degrees
- moved J1 20.5 mm to (133.1, 86.7), turned to 270 degrees
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Connections:
- net VCC renamed +6V
- JP1 pad 1: Net-(C1-Pad2) -> Net-(J1-Pad1)
- JP1 pad 2: Net-(J1-Pad1) -> Net-(C1-Pad2)
Routing:
- net +6V: track 0.00 -> 73.7 mm, vias 0 -> 2
- net Net-(JP4-Pad1): track 0.00 -> 29.6 mm
- net Net-(C1-Pad1): track 0.00 -> 29.1 mm
- net Net-(J3-Pad1): track 5.75 -> 31.4 mm
- net GND: track 0.00 -> 21.5 mm, vias 0 -> 4
- net Net-(D2-Pad2): track 0.00 -> 13.8 mm
- net Net-(U1-Pad12): track 0.00 -> 13.2 mm
- net Net-(C1-Pad2): track 0.00 -> 11.2 mm
- net Net-(U1-Pad13): track 0.00 -> 10.9 mm
- net Net-(C2-Pad2): track 0.00 -> 10.1 mm
- net Net-(U1-Pad11): track 0.00 -> 8.58 mm
- net Net-(J1-Pad1): track 0.00 -> 5.19 mm
- net Net-(JP5-Pad2): track 0.00 -> 3.46 mm
- net Net-(JP4-Pad2): track 0.00 -> 3.46 mm
- net Net-(D1-Pad2): track 0.00 -> 3.30 mm
- added copper zone on B.Cu, net GND
Other:
- board outline added: 82.5 x 69.8 mm

Commit message: Complete layout. Just need to finalize microstrip length
Parts:
- moved D2 7.62 mm to (180.6, 65.8)
- moved U1 0.13 mm to (165.4, 89.7)
Routing:
- net Net-(U1-Pad13): track 10.9 -> 0.54 mm
- net Net-(D2-Pad2): track 13.8 -> 6.22 mm
- net GND: track 21.5 -> 14.5 mm, vias 4 -> 5
- net Net-(U1-Pad12): track 13.2 -> 8.39 mm
- net +6V: track 73.7 -> 75.5 mm

Commit message: added new HC00 Footprint under digikey.pretty
Parts:
- J3: footprint My_Footprints:Vertical_BNC_Connector -> My_Footprints:BNC_Connector
- moved J4 90.2 mm to (118.8, 112.2), turned to 0 degrees
- moved J1 70.3 mm to (197.1, 57.8), turned to 180 degrees
- moved JP1 66.2 mm to (199.6, 62.0), turned to 180 degrees
- moved JP2 63.5 mm to (194.6, 62.0), turned to 180 degrees
- moved C1 53.1 mm to (194.6, 68.7)
- moved D1 53.0 mm to (137.0, 92.4), turned to 90 degrees
- moved R1 49.6 mm to (202.9, 98.1)
- moved J3 48.3 mm to (222.0, 112.2)
- moved C2 44.0 mm to (143.1, 93.4), turned to 90 degrees
- moved R2 40.1 mm to (194.6, 88.3), turned to 270 degrees
- moved R7 39.5 mm to (222.0, 106.4), turned to 90 degrees
- moved R3 36.5 mm to (157.6, 96.1), turned to 270 degrees
- moved U1 35.2 mm to (194.6, 109.3), turned to 0 degrees
- moved J2 35.0 mm to (137.0, 78.9), turned to 180 degrees
- moved U2 33.7 mm to (148.2, 86.1), turned to 0 degrees
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Connections:
- JP3 pad 1: GND -> Net-(J3-Pad1)
- JP3 pad 2: Net-(J3-Pad1) -> GND
- U1 pad 1: Net-(C1-Pad1) -> Net-(U1-Pad1)
- U1 pad 10: +6V -> Net-(C1-Pad1)
- U1 pad 12: Net-(U1-Pad12) -> Net-(U1-Pad1)
- U1 pad 13: Net-(U1-Pad13) -> +6V
- U1 pad 2: Net-(C1-Pad1) -> Net-(U1-Pad11)
- U1 pad 3: Net-(U1-Pad12) -> Net-(U1-Pad3)
- U1 pad 4: Net-(U1-Pad11) -> Net-(U1-Pad3)
- U1 pad 5: Net-(U1-Pad11) -> Net-(U1-Pad3)
- U1 pad 8: Net-(U1-Pad13) -> Net-(U1-Pad1)
- U1 pad 9: Net-(U1-Pad12) -> Net-(C1-Pad1)
Routing:
- net Net-(J4-Pad1): track 0.00 -> 211.0 mm
- net Net-(C1-Pad1): track 29.1 -> 45.3 mm
- net Net-(U1-Pad1): track 0.00 -> 15.9 mm
- net GND: track 14.5 -> 0.00 mm, vias 5 -> 7
- net Net-(JP4-Pad1): track 29.6 -> 15.3 mm
- net Net-(U1-Pad12): track 8.39 -> 0.00 mm
- net +6V: track 75.5 -> 67.9 mm, vias 2 -> 0
- net Net-(J3-Pad1): track 31.4 -> 28.2 mm
- net Net-(C1-Pad2): track 11.2 -> 8.21 mm
- net Net-(U1-Pad3): track 0.00 -> 2.54 mm
- net Net-(D2-Pad2): track 6.22 -> 8.51 mm
- net Net-(C2-Pad2): track 10.1 -> 10.9 mm
- net Net-(U1-Pad13): track 0.54 -> 0.00 mm
- added copper zone on F.Cu, net GND
- removed copper zone on F.Cu, net Net-(J4-Pad1)
Other:
- board size 82.5 x 69.8 mm -> 127 x 75.3 mm
- rule trace_min: 0.2 -> 1.27
- rule via_min_size: 0.4 -> 0.508

Commit message: pushed to pull. no changes
Parts:
- U1: footprint My_Footprints:HC00 -> digikey:SN74HC00DR
- moved U1 6.33 mm to (198.3, 104.2), turned to 90 degrees
Routing:
- net Net-(U1-Pad11): track 8.36 -> 5.98 mm
- net Net-(U1-Pad1): track 15.9 -> 13.8 mm
- net Net-(C1-Pad1): track 45.3 -> 43.8 mm
- net Net-(JP4-Pad1): track 15.3 -> 14.5 mm
- net +6V: track 67.9 -> 67.3 mm
Other:
- rule trace_min: 1.27 -> 0.24638
