File: EE173/Summer/EE173_Lab4.kicad_pcb (KiCad board)
At the start: 2 copper layers, 26 parts, among them J1 Conn_01x02_Male, J2 Conn_01x02_Male, J3 Conn_Coaxial, J4 Conn_Coaxial, U1 74HC00, U2 L7806, U4 50ohm

Commit message: nothing changed
Parts:
- removed R4: R, Resistor_SMD:R_0805_2012Metric
- removed U4: 50ohm, My_Footprints:MicroStrip
- J1, J2, JP1, JP2, JP3, JP4, JP5, JP6: footprint My_Footprints:Two_Pos_Jumper -> My_Footprints:header_2_pins
- J3: value Conn_Coaxial -> Test Line; footprint My_Footprints:BNC_Connector -> My_Footprints:Vertical_BNC_Connector
- J4: value Conn_Coaxial -> OSC
- moved J4 90.6 mm to (234.3, 23.3), turned to 180 degrees
- moved JP4 77.3 mm to (213.2, 37.3)
- moved JP2 77.0 mm to (198.6, 31.0), turned to 270 degrees
- moved J1 76.4 mm to (188.0, 25.4), turned to 90 degrees
- moved JP1 72.5 mm to (188.0, 31.0), turned to 270 degrees
- moved R7 70.7 mm to (234.3, 45.1), turned to 90 degrees
- moved JP5 61.4 mm to (213.1, 45.5)
- moved R2 60.4 mm to (193.4, 40.1), turned to 180 degrees
- moved R5 59.4 mm to (224.1, 39.1), turned to 180 degrees
- moved C3 58.1 mm to (199.9, 48.4), turned to 90 degrees
- moved C4 58.0 mm to (203.2, 48.4), turned to 90 degrees
- moved JP6 57.4 mm to (213.1, 52.9)
- moved C1 57.2 mm to (189.0, 43.3), turned to 180 degrees
- moved J3 55.2 mm to (234.3, 51.5), turned to 180 degrees
- moved R3 54.5 mm to (196.6, 48.4), turned to 90 degrees
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Connections:
- C3 pad 2: VCC -> +6V
- C4 pad 2: VCC -> +6V
- JP3 pad 1: Net-(JP3-Pad1) -> GND
- JP3 pad 2: Net-(JP3-Pad2) -> Net-(J3-Pad1)
- JP4 pad 1: Net-(JP3-Pad1) -> Net-(JP4-Pad1)
- JP5 pad 1: Net-(JP3-Pad1) -> Net-(JP4-Pad1)
- JP6 pad 1: Net-(JP3-Pad1) -> Net-(JP4-Pad1)
- JP6 pad 2: Net-(JP6-Pad2) -> Net-(J3-Pad1)
- R1 pad 1: VCC -> +6V
- R3 pad 2: VCC -> +6V
- R5 pad 1: Net-(JP6-Pad2) -> Net-(J3-Pad1)
- R6 pad 1: Net-(JP6-Pad2) -> Net-(J3-Pad1)
- R7 pad 1: Net-(JP6-Pad2) -> Net-(J3-Pad1)
- R7 pad 2: Net-(J3-Pad1) -> Net-(J4-Pad1)
- U1 pad 1: Net-(C1-Pad1) -> Net-(U1-Pad1)
- U1 pad 10: VCC -> Net-(C1-Pad1)
- U1 pad 12: Net-(U1-Pad12) -> Net-(U1-Pad1)
- U1 pad 13: Net-(U1-Pad13) -> +6V
- U1 pad 14: VCC -> +6V
- U1 pad 2: Net-(C1-Pad1) -> Net-(U1-Pad11)
- U1 pad 3: Net-(U1-Pad12) -> Net-(U1-Pad3)
- U1 pad 4: Net-(U1-Pad11) -> Net-(U1-Pad3)
- U1 pad 5: Net-(U1-Pad11) -> Net-(U1-Pad3)
- U1 pad 6: Net-(JP3-Pad1) -> Net-(JP4-Pad1)
- U1 pad 8: Net-(U1-Pad13) -> Net-(U1-Pad1)
- U1 pad 9: Net-(U1-Pad12) -> Net-(C1-Pad1)
- U2 pad 3: VCC -> +6V
Routing:
- net Net-(J3-Pad1): track 0.00 -> 47.1 mm
- net Net-(JP4-Pad1): track 0.00 -> 25.4 mm
- net Net-(C1-Pad2): track 0.00 -> 20.5 mm
- net +6V: track 0.00 -> 20.1 mm
- net Net-(J4-Pad1): track 0.00 -> 19.7 mm
- net Net-(C2-Pad2): track 0.00 -> 12.1 mm
- net Net-(C1-Pad1): track 0.00 -> 11.3 mm
- net Net-(JP5-Pad2): track 0.00 -> 9.47 mm
- net Net-(JP4-Pad2): track 0.00 -> 9.46 mm
- net Net-(U1-Pad1): track 0.00 -> 8.90 mm
- net Net-(U1-Pad11): track 0.00 -> 8.90 mm
- net Net-(D2-Pad2): track 0.00 -> 6.22 mm
- net Net-(D1-Pad2): track 0.00 -> 5.69 mm
- net Net-(J1-Pad1): track 0.00 -> 5.59 mm
- net Net-(U1-Pad3): track 0.00 -> 3.62 mm
- added copper zone on B.Cu, net GND
- added copper zone on F.Cu, net GND
Other:
- board outline added: 55.9 x 43.2 mm
- rule trace_min: 0.2 -> 0.24638
- rule via_min_size: 0.4 -> 0.508

Commit message: updated header 2 pins
Parts:
- U1: footprint My_Footprints:HC00 -> digikey:SN74HC00DR
- moved U1 3.57 mm to (202.1, 40.9), turned to 180 degrees
- moved R2 3.00 mm to (195.6, 38.1)
Routing:
- net Net-(C1-Pad1): track 11.3 -> 20.4 mm
- net Net-(U1-Pad1): track 8.90 -> 13.0 mm
- net Net-(U1-Pad11): track 8.90 -> 5.98 mm
- net +6V: track 20.1 -> 23.0 mm
- net Net-(U1-Pad3): track 3.62 -> 2.54 mm
- net Net-(JP4-Pad1): track 25.4 -> 24.8 mm
