File: EE173/Summer/EE173_Lab4.sch (KiCad schematic (older format))
At the start: 24 parts, among them J1 Conn_01x02_Male, J2 Conn_01x02_Male, J3 Test Line, J4 OSC, U1 74HC00, U2 L7806

Commit message: made header 2 pins
Parts:
- D2: footprint LED_SMD:LED_0805_2012Metric -> LED_THT:LED_D5.0mm
- J4: footprint Connector_Coaxial:BNC_PanelMountable_Vertical -> My_Footprints:BNC_Connector
Changed lines of the file:
@@
 F 0 "J4" H 9549 5726 50  0000 L CNN
 F 1 "OSC" H 9549 5635 50  0000 L CNN
-F 2 "Connector_Coaxial:BNC_PanelMountable_Vertical" H 9450 5750 50  0001 C CNN
+F 2 "My_Footprints:BNC_Connector" H 9450 5750 50  0001 C CNN
 F 3 " ~" H 9450 5750 50  0001 C CNN
 	1    9450 5750
@@
 F 0 "D2" H 6392 1745 50  0000 C CNN
 F 1 "LED" H 6392 1836 50  0000 C CNN
-F 2 "LED_SMD:LED_0805_2012Metric" H 6400 2000 50  0001 C CNN
+F 2 "LED_THT:LED_D5.0mm" H 6400 2000 50  0001 C CNN
 F 3 "~" H 6400 2000 50  0001 C CNN
 	1    6400 2000

Commit message: nothing changed
Parts:
- J1, J2: footprint Connector_Pin:Pin_D0.7mm_L6.5mm_W1.8mm_FlatFork -> My_Footprints:header_2_pins
- JP1, JP2, JP3, JP4, JP5, JP6: footprint Jumper:SolderJumper-2_P1.3mm_Bridged2Bar_Pad1.0x1.5mm -> My_Footprints:header_2_pins
Connections:
- net at C1.1, R1.2, R2.1: now also U1.10, U1.9; no longer U1.1, U1.2
- net at JP3.2, JP6.2, R5.1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: now also J3.1 (In)
- net at J4.1 (In), R7.2: no longer J3.1 (In)
- net at U1.4, U1.5: now also U1.3; no longer U1.11
- net at U1.8: now also U1.1, U1.12; no longer U1.13
- net VCC renamed +6V
- net +6V: now also U1.13; no longer U1.10
- new net: U1.11, U1.2
Other:
- moved on the sheet: C1, J1, J3, J4, JP1, JP2, JP3, JP4, JP5, JP6, R1, R2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

Commit message: header 2 pins hole size to 1.02mm
Parts:
- U1: footprint My_Footprints:HC00 -> digikey:SN74HC00DR
Changed lines of the file:
@@
 F 0 "U1" H 6000 4725 50  0000 C CNN
 F 1 "74HC00" H 6000 4634 50  0000 C CNN
-F 2 "My_Footprints:HC00" H 6000 4400 50  0001 C CNN
+F 2 "digikey:SN74HC00DR" H 6000 4400 50  0001 C CNN
 F 3 "http://www.ti.com/lit/gpn/sn74hc00" H 6000 4400 50  0001 C CNN
 	1    6000 4400
@@
 F 0 "U1" H 7050 4725 50  0000 C CNN
 F 1 "74HC00" H 7050 4634 50  0000 C CNN
-F 2 "My_Footprints:HC00" H 7050 4400 50  0001 C CNN
+F 2 "digikey:SN74HC00DR" H 7050 4400 50  0001 C CNN
 F 3 "http://www.ti.com/lit/gpn/sn74hc00" H 7050 4400 50  0001 C CNN
 	2    7050 4400
@@
 F 0 "U1" H 4350 4575 50  0000 C CNN
 F 1 "74HC00" H 4350 4484 50  0000 C CNN
-F 2 "My_Footprints:HC00" H 4350 4250 50  0001 C CNN
+F 2 "digikey:SN74HC00DR" H 4350 4250 50  0001 C CNN
 F 3 "http://www.ti.com/lit/gpn/sn74hc00" H 4350 4250 50  0001 C CNN
 	3    4350 4250
@@
 F 0 "U1" H 5200 5125 50  0000 C CNN
 F 1 "74HC00" H 5200 5034 50  0000 C CNN
-F 2 "My_Footprints:HC00" H 5200 4800 50  0001 C CNN
+F 2 "digikey:SN74HC00DR" H 5200 4800 50  0001 C CNN
 F 3 "http://www.ti.com/lit/gpn/sn74hc00" H 5200 4800 50  0001 C CNN
 	4    5200 4800
@@
 F 0 "U1" H 5880 3296 50  0000 L CNN
 F 1 "74HC00" H 5880 3205 50  0000 L CNN
-F 2 "My_Footprints:HC00" H 5650 3250 50  0001 C CNN
+F 2 "digikey:SN74HC00DR" H 5650 3250 50  0001 C CNN
 F 3 "http://www.ti.com/lit/gpn/sn74hc00" H 5650 3250 50  0001 C CNN
 	5    5650 3250
