File: EE173/Conner/EE173_Lab4.kicad_pcb (KiCad board)
At the start: 2 copper layers, 26 parts, among them J1 Conn_01x02_Male, J2 Conn_01x02_Male, J3 Conn_Coaxial, J4 Conn_Coaxial, U1 74HC00, U2 L7806, U4 50ohm

Commit message: Not new added
Parts:
- removed R4: R, Resistor_SMD:R_0805_2012Metric
- removed U4: 50ohm, My_Footprints:MicroStrip
- J1, J2, JP1, JP2, JP3, JP4, JP5, JP6: footprint My_Footprints:Two_Pos_Jumper -> My_Footprints:header_2_pins
- J3: value Conn_Coaxial -> Test Line; footprint My_Footprints:BNC_Connector -> My_Footprints:Vertical_BNC_Connector
- J4: value Conn_Coaxial -> OSC
- moved J4 105.5 mm to (281.0, 62.9), turned to 90 degrees
- moved JP2 103.5 mm to (241.5, 28.4), turned to 90 degrees
- moved J1 103.5 mm to (237.8, 19.9)
- moved JP1 97.6 mm to (237.0, 28.6), turned to 90 degrees
- moved JP4 83.1 mm to (248.4, 77.8)
- moved R7 82.0 mm to (264.8, 62.9)
- moved C1 79.7 mm to (239.4, 38.2), turned to 90 degrees
- moved JP6 74.7 mm to (248.4, 68.9)
- moved J3 71.6 mm to (259.4, 62.9), turned to 270 degrees
- moved R2 71.3 mm to (245.3, 52.0)
- moved JP3 69.6 mm to (248.3, 73.2)
- moved C4 69.4 mm to (234.6, 58.1), turned to 270 degrees
- moved JP5 66.1 mm to (248.5, 82.7)
- moved J2 64.0 mm to (189.6, 37.6)
- moved R5 56.8 mm to (255.9, 77.9), turned to 180 degrees
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Connections:
- net VCC renamed +6V
- JP3 pad 1: Net-(JP3-Pad1) -> GND
- JP3 pad 2: Net-(JP3-Pad2) -> Net-(J3-Pad1)
- JP4 pad 1: Net-(JP3-Pad1) -> Net-(JP4-Pad1)
- JP5 pad 1: Net-(JP3-Pad1) -> Net-(JP4-Pad1)
- JP6 pad 1: Net-(JP3-Pad1) -> Net-(JP4-Pad1)
- JP6 pad 2: Net-(JP6-Pad2) -> Net-(J3-Pad1)
- R5 pad 1: Net-(JP6-Pad2) -> Net-(J3-Pad1)
- R6 pad 1: Net-(JP6-Pad2) -> Net-(J3-Pad1)
- R7 pad 1: Net-(JP6-Pad2) -> Net-(J3-Pad1)
- R7 pad 2: Net-(J3-Pad1) -> Net-(J4-Pad1)
- U1 pad 6: Net-(JP3-Pad1) -> Net-(JP4-Pad1)
Routing:
- net Net-(J3-Pad1): track 0.00 -> 48.7 mm
- net +6V: track 0.00 -> 38.3 mm
- net Net-(JP4-Pad1): track 0.00 -> 30.0 mm
- net Net-(U1-Pad12): track 0.00 -> 22.9 mm, vias 0 -> 2
- net Net-(U1-Pad13): track 0.00 -> 11.3 mm
- net Net-(U1-Pad11): track 0.00 -> 8.58 mm
- net Net-(D2-Pad2): track 0.00 -> 3.81 mm
- net Net-(C1-Pad1): track 0.00 -> 1.27 mm
- added copper zone on F.Cu, net Net-(J4-Pad1)

Commit message: Finished Layout
Parts:
- moved J4 35.2 mm to (259.4, 35.1), turned to 180 degrees
- moved J1 19.5 mm to (236.6, 39.4), turned to 270 degrees
- moved JP1 11.1 mm to (239.6, 39.4), turned to 270 degrees
- moved JP2 11.1 mm to (242.9, 39.4), turned to 270 degrees
- moved R7 8.06 mm to (259.4, 56.9), turned to 90 degrees
- moved C1 7.59 mm to (239.6, 45.8)
- moved R2 3.84 mm to (248.3, 54.3)
- moved R1 2.41 mm to (238.6, 54.3)
- moved C4 2.10 mm to (233.7, 59.9), turned to 90 degrees
- moved J2 1.56 mm to (190.0, 39.1)
- moved U2 0.77 mm to (200.0, 57.6)
- moved D1 0.64 mm to (190.0, 53.1)
- moved C2 0.41 mm to (190.0, 60.1)
- moved R6 0.13 mm to (255.9, 82.7)
Connections:
- U1 pad 1: Net-(C1-Pad1) -> Net-(U1-Pad1)
- U1 pad 10: +6V -> Net-(C1-Pad1)
- U1 pad 12: Net-(U1-Pad12) -> Net-(U1-Pad1)
- U1 pad 13: Net-(U1-Pad13) -> +6V
- U1 pad 2: Net-(C1-Pad1) -> Net-(U1-Pad11)
- U1 pad 3: Net-(U1-Pad12) -> Net-(U1-Pad3)
- U1 pad 4: Net-(U1-Pad11) -> Net-(U1-Pad3)
- U1 pad 5: Net-(U1-Pad11) -> Net-(U1-Pad3)
- U1 pad 8: Net-(U1-Pad13) -> Net-(U1-Pad1)
- U1 pad 9: Net-(U1-Pad12) -> Net-(C1-Pad1)
Routing:
- net Net-(C1-Pad1): track 1.27 -> 28.0 mm
- net Net-(U1-Pad12): track 22.9 -> 0.00 mm, vias 2 -> 0
- net Net-(J4-Pad1): track 0.00 -> 19.6 mm
- net Net-(U1-Pad1): track 0.00 -> 17.2 mm
- net Net-(U1-Pad13): track 11.3 -> 0.00 mm
- net Net-(C2-Pad2): track 0.00 -> 11.0 mm
- net +6V: track 38.3 -> 45.0 mm
- net Net-(C1-Pad2): track 0.00 -> 6.26 mm
- net Net-(JP4-Pad2): track 0.00 -> 3.99 mm
- net Net-(JP5-Pad2): track 0.00 -> 3.92 mm
- net Net-(D1-Pad2): track 0.00 -> 3.81 mm
- net Net-(J1-Pad1): track 0.00 -> 3.04 mm
- net Net-(U1-Pad3): track 0.00 -> 2.54 mm
- net GND: vias 0 -> 7
- added copper zone on B.Cu, net GND
- added copper zone on F.Cu, net GND
- removed copper zone on F.Cu, net Net-(J4-Pad1)
Other:
- board outline added: 81.3 x 57.1 mm
- rule trace_min: 0.2 -> 0.24638
- rule via_min_size: 0.4 -> 0.508

Commit message: Nothing New
Parts:
- U1: footprint My_Footprints:HC00 -> digikey:SN74HC00DR
- moved U1 5.37 mm to (241.5, 61.4), turned to 90 degrees
Routing:
- net Net-(JP4-Pad1): track 29.9 -> 32.4 mm
- net Net-(U1-Pad11): track 8.36 -> 5.98 mm
- net Net-(U1-Pad1): track 17.2 -> 14.8 mm

Commit message: Changed Schematic
Put all three circuits in the same schematic and added coax connectors
Parts:
- J3: footprint My_Footprints:Vertical_BNC_Connector -> Connector_Coaxial:SMA_Amphenol_132289_EdgeMount
- J4: footprint My_Footprints:BNC_Connector -> Connector_Coaxial:SMA_Amphenol_132289_EdgeMount
- moved J2 77.5 mm to (212.8, 113.2), turned to 90 degrees
- moved D1 70.6 mm to (227.1, 113.2), turned to 180 degrees
- moved C2 69.0 mm to (234.1, 113.2), turned to 180 degrees
- moved U2 55.5 mm to (231.6, 103.2), turned to 90 degrees
- moved C3 48.6 mm to (233.8, 98.6), turned to 180 degrees
- moved D2 41.3 mm to (224.7, 90.2), turned to 0 degrees
- moved R3 37.5 mm to (232.0, 90.2), turned to 0 degrees
- moved JP2 36.1 mm to (213.4, 60.3), turned to 0 degrees
- moved J1 35.9 mm to (213.4, 66.9), turned to 0 degrees
- moved JP1 35.6 mm to (213.4, 63.5), turned to 0 degrees
- moved C1 26.6 mm to (219.8, 63.6), turned to 180 degrees
- moved JP3 22.0 mm to (245.2, 51.5)
- moved R2 20.0 mm to (228.3, 54.8), turned to 90 degrees
- moved JP4 14.7 mm to (245.2, 63.5)
- moved R5 14.6 mm to (252.7, 63.6)
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Routing:
- net Net-(J3-Pad1): track 48.9 -> 42.0 mm
- net Net-(JP4-Pad1): track 32.4 -> 27.0 mm
- net GND: track 0.00 -> 0.96 mm, vias 7 -> 6
- net +6V: track 45.0 -> 44.2 mm
Other:
- board size 81.3 x 57.1 mm -> 59.4 x 88.9 mm
- net class Default: clearance 0.2 -> 0.254; trace_width 0.25 -> 0.254; via_dia 0.8 -> 0.889; via_drill 0.4 -> 0.508
- net class Power added: clearance 0.254, trace_width 1.27, via_dia 0.889, via_drill 0.508
- rule trace_clearance: 0.2 -> 0.254
- rule trace_min: 0.24638 -> 0.254
- board text added: "+ -"
- board text added: "CH REV0"
- board text added: "Osc"
- board text added: "Test Line"
- board text added: "sig"
