File: EE173/Conner/EE173_Lab4.sch (KiCad schematic (older format))
At the start: 24 parts, among them J1 Conn_01x02_Male, J2 Conn_01x02_Male, J3 Test Line, J4 OSC, U1 74HC00, U2 L7806

Commit message: Edited HC00 footprint
Parts:
- D2: footprint LED_SMD:LED_0805_2012Metric -> LED_THT:LED_D5.0mm
Other:
- note added: "50ohm Microstrip"
Changed lines of the file:
@@
 F 0 "D2" H 6392 1745 50  0000 C CNN
 F 1 "LED" H 6392 1836 50  0000 C CNN
-F 2 "LED_SMD:LED_0805_2012Metric" H 6400 2000 50  0001 C CNN
+F 2 "LED_THT:LED_D5.0mm" H 6400 2000 50  0001 C CNN
 F 3 "~" H 6400 2000 50  0001 C CNN
 	1    6400 2000
@@
 Wire Wire Line
 	8850 5050 8850 5750
+Wire Notes Line
+	8750 5200 8750 5650
+Wire Notes Line
+	8750 5650 8950 5650
+Wire Notes Line
+	8950 5650 8950 5200
+Wire Notes Line
+	8750 5200 8950 5200
+Text Notes 8700 5750 1    50   ~ 0
+50ohm Microstrip
 $EndSCHEMATC

Commit message: Made no changes
Parts:
- J1, J2: footprint Connector_Pin:Pin_D0.7mm_L6.5mm_W1.8mm_FlatFork -> My_Footprints:header_2_pins
- JP1, JP2, JP3, JP4, JP5, JP6: footprint Jumper:SolderJumper-2_P1.3mm_Bridged2Bar_Pad1.0x1.5mm -> My_Footprints:header_2_pins
Changed lines of the file:
@@
 F 0 "J1" H 2256 3828 50  0000 C CNN
 F 1 "Conn_01x02_Male" H 2256 3737 50  0000 C CNN
-F 2 "Connector_Pin:Pin_D0.7mm_L6.5mm_W1.8mm_FlatFork" H 2150 3650 50  0001 C CNN
+F 2 "My_Footprints:header_2_pins" H 2150 3650 50  0001 C CNN
 F 3 "~" H 2150 3650 50  0001 C CNN
 	1    2150 3650
@@
 F 0 "J2" H 3756 2178 50  0000 C CNN
 F 1 "Conn_01x02_Male" H 3350 2100 50  0000 C CNN
-F 2 "Connector_Pin:Pin_D0.7mm_L6.5mm_W1.8mm_FlatFork" H 3650 2000 50  0001 C CNN
+F 2 "My_Footprints:header_2_pins" H 3650 2000 50  0001 C CNN
 F 3 "~" H 3650 2000 50  0001 C CNN
 	1    3650 2000
@@
 F 0 "JP3" H 7900 4014 50  0000 C CNN
 F 1 "Jumper" H 7900 3923 50  0000 C CNN
-F 2 "Jumper:SolderJumper-2_P1.3mm_Bridged2Bar_Pad1.0x1.5mm" H 7900 3750 50  0001 C CNN
+F 2 "My_Footprints:header_2_pins" H 7900 3750 50  0001 C CNN
 F 3 "~" H 7900 3750 50  0001 C CNN
 	1    7900 3750
@@
 F 0 "JP4" H 7900 4364 50  0000 C CNN
 F 1 "Jumper" H 7900 4273 50  0000 C CNN
-F 2 "Jumper:SolderJumper-2_P1.3mm_Bridged2Bar_Pad1.0x1.5mm" H 7900 4100 50  0001 C CNN
+F 2 "My_Footprints:header_2_pins" H 7900 4100 50  0001 C CNN
 F 3 "~" H 7900 4100 50  0001 C CNN
 	1    7900 4100
@@
 F 0 "JP5" H 7900 4714 50  0000 C CNN
 F 1 "Jumper" H 7900 4623 50  0000 C CNN
-F 2 "Jumper:SolderJumper-2_P1.3mm_Bridged2Bar_Pad1.0x1.5mm" H 7900 4450 50  0001 C CNN
+F 2 "My_Footprints:header_2_pins" H 7900 4450 50  0001 C CNN
 F 3 "~" H 7900 4450 50  0001 C CNN
 	1    7900 4450
@@
 F 0 "JP6" H 7900 4450 50  0000 C CNN
 F 1 "Jumper" H 7900 4550 50  0000 C CNN
-F 2 "Jumper:SolderJumper-2_P1.3mm_Bridged2Bar_Pad1.0x1.5mm" H 7900 4650 50  0001 C CNN
+F 2 "My_Footprints:header_2_pins" H 7900 4650 50  0001 C CNN
 F 3 "~" H 7900 4650 50  0001 C CNN
 	1    7900 4650
@@
 F 0 "JP1" H 3150 4350 50  0000 C CNN
 F 1 "Jumper" H 3150 4450 50  0000 C CNN
-F 2 "Jumper:SolderJumper-2_P1.3mm_Bridged2Bar_Pad1.0x1.5mm" H 3150 4200 50  0001 C CNN
+F 2 "My_Footprints:header_2_pins" H 3150 4200 50  0001 C CNN
 F 3 "~" H 3150 4200 50  0001 C CNN
 	1    3150 4200
@@
 F 0 "JP2" H 3150 4200 50  0000 C CNN
 F 1 "Jumper" H 3150 4300 50  0000 C CNN
-F 2 "Jumper:SolderJumper-2_P1.3mm_Bridged2Bar_Pad1.0x1.5mm" H 3150 4400 50  0001 C CNN
+F 2 "My_Footprints:header_2_pins" H 3150 4400 50  0001 C CNN
 F 3 "~" H 3150 4400 50  0001 C CNN
 	1    3150 4400

Commit message: Vertical BNC Footprint
Parts:
- J4: footprint Connector_Coaxial:BNC_PanelMountable_Vertical -> My_Footprints:BNC_Connector
Changed lines of the file:
@@
 F 0 "J4" H 9549 5726 50  0000 L CNN
 F 1 "OSC" H 9549 5635 50  0000 L CNN
-F 2 "Connector_Coaxial:BNC_PanelMountable_Vertical" H 9450 5750 50  0001 C CNN
+F 2 "My_Footprints:BNC_Connector" H 9450 5750 50  0001 C CNN
 F 3 " ~" H 9450 5750 50  0001 C CNN
 	1    9450 5750

Commit message: Not new added
Connections:
- net at JP3.2, JP6.2, R5.1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: now also J3.1 (In)
- net at J4.1 (In), R7.2: no longer J3.1 (In)
- net VCC renamed +6V
Other:
- moved on the sheet: J3, R7
Changed lines of the file:
@@
 Connection ~ 3900 4300
-$Comp
-L power:VCC #PWR08
-U 1 1 5BF3574A
-P 5000 4950
-F 0 "#PWR08" H 5000 4800 50  0001 C CNN
-F 1 "VCC" V 5018 5077 50  0000 L CNN
-F 2 "" H 5000 4950 50  0001 C CNN
-F 3 "" H 5000 4950 50  0001 C CNN
-	1    5000 4950
-	0    -1   -1   0
-$EndComp
 $Comp
 L Device:R R7
 U 1 1 5BF35A5D
-P 8850 4850
-F 0 "R7" H 8920 4896 50  0000 L CNN
-F 1 "R" H 8920 4805 50  0000 L CNN
-F 2 "Resistor_SMD:R_0805_2012Metric" V 8780 4850 50  0001 C CNN
-F 3 "~" H 8850 4850 50  0001 C CNN
-	1    8850 4850
-	1    0    0    -1
-$EndComp
-Wire Wire Line
-	8850 5000 8850 5050
+P 8850 5200
+F 0 "R7" H 8920 5246 50  0000 L CNN
+F 1 "R" H 8920 5155 50  0000 L CNN
+F 2 "Resistor_SMD:R_0805_2012Metric" V 8780 5200 50  0001 C CNN
+F 3 "~" H 8850 5200 50  0001 C CNN
+	1    8850 5200
+	1    0    0    -1
+$EndComp
 $Comp
 L EE173_Lab4-rescue:Conn_Coaxial-My_Connector J3
 U 1 1 5BF5C810
-P 9450 5050
-F 0 "J3" H 9549 5026 50  0000 L CNN
-F 1 "Test Line" H 9549 4935 50  0000 L CNN
-F 2 "My_Footprints:Vertical_BNC_Connector" H 9450 5050 50  0001 C CNN
-F 3 " ~" H 9450 5050 50  0001 C CNN
-	1    9450 5050
-	1    0    0    -1
-$EndComp
-Connection ~ 8850 5050
+P 9450 4750
+F 0 "J3" H 9549 4726 50  0000 L CNN
+F 1 "Test Line" H 9549 4635 50  0000 L CNN
+F 2 "My_Footprints:Vertical_BNC_Connector" H 9450 4750 50  0001 C CNN
+F 3 " ~" H 9450 4750 50  0001 C CNN
+	1    9450 4750
+	1    0    0    -1
+$EndComp
 $Comp
 L power:GND #PWR014
 U 1 1 5BF5C968
-P 9450 5350
-F 0 "#PWR014" H 9450 5100 50  0001 C CNN
-F 1 "GND" H 9455 5177 50  0000 C CNN
-F 2 "" H 9450 5350 50  0001 C CNN
-F 3 "" H 9450 5350 50  0001 C CNN
-	1    9450 5350
-	1    0    0    -1
-$EndComp
-Wire Wire Line
-	9450 5350 9450 5250
-Wire Wire Line
-	8850 5050 9250 5050
+P 9450 5050
+F 0 "#PWR014" H 9450 4800 50  0001 C CNN
+F 1 "GND" H 9455 4877 50  0000 C CNN
+F 2 "" H 9450 5050 50  0001 C CNN
+F 3 "" H 9450 5050 50  0001 C CNN
+	1    9450 5050
+	1    0    0    -1
+$EndComp
+Wire Wire Line
+	9450 5050 9450 4950
+Wire Wire Line
+	8850 4750 9250 4750
 $Comp
 L EE173_Lab4-rescue:Conn_Coaxial-My_Connector J4
@@
 	8850 5750 9250 5750
 $Comp
-L Regulator_Linear:L7806 U2
-U 1 1 5BF5D575
-P 4850 2000
-F 0 "U2" H 4850 2242 50  0000 C CNN
-F 1 "L7806" H 4850 2151 50  0000 C CNN
-F 2 "My_Footprints:L7806ABV" H 4875 1850 50  0001 L CIN
-F 3 "http://www.st.com/content/ccc/resource/technical/document/datasheet/41/4f/b3/b0/12/d4/47/88/CD00000444.pdf/files/CD00000444.pdf/jcr:content/translations/en.CD00000444.pdf" H 4850 1950 50  0001 C CNN
-	1    4850 2000
-	1    0    0    -1
-$EndComp
-$Comp
 L 74xx:74HC00 U1
 U 1 1 5BF5D5E6
@@
 Wire Wire Line
 	5200 4300 5950 4300
-Wire Wire Line
-	5000 4950 5200 4950
 Wire Wire Line
 	4500 4200 4500 4300
@@
 	1    0    0    -1
 $EndComp
-$Comp
-L power:VCC #PWR09
-U 1 1 5BF65AF9
-P 5250 1900
-F 0 "#PWR09" H 5250 1750 50  0001 C CNN
-F 1 "VCC" H 5267 2073 50  0000 C CNN
-F 2 "" H 5250 1900 50  0001 C CNN
-F 3 "" H 5250 1900 50  0001 C CNN
-	1    5250 1900
-	1    0    0    -1
-$EndComp
 Wire Wire Line
 	5150 2000 5250 2000
-Wire Wire Line
-	5250 2000 5250 1900
 Connection ~ 5250 2000
 Wire Wire Line
@@
 	8200 4450 8350 4450
 Wire Wire Line
-	8850 4700 8850 4650
-Wire Wire Line
 	8650 4100 8850 4100
 Connection ~ 8850 4100
@@
 Connection ~ 3500 4300
 $Comp
-L power:VCC #PWR04
-U 1 1 5BFCFBE7
-P 3900 3750
-F 0 "#PWR04" H 3900 3600 50  0001 C CNN
-F 1 "VCC" V 3918 3877 50  0000 L CNN
-F 2 "" H 3900 3750 50  0001 C CNN
-F 3 "" H 3900 3750 50  0001 C CNN
-	1    3900 3750
-	1    0    0    -1
-$EndComp
-Wire Wire Line
-	3900 3950 3900 3750
-$Comp
 L power:GND #PWR05
 U 1 1 5BFD3FF6
@@
 	7450 3750 7450 3850
 Wire Wire Line
-	8850 5050 8850 5750
-Wire Notes Line
-	8750 5200 8750 5650
-Wire Notes Line
-	8750 5650 8950 5650
-Wire Notes Line
-	8950 5650 8950 5200
-Wire Notes Line
-	8750 5200 8950 5200
-Text Notes 8700 5750 1    50   ~ 0
+	8850 4650 8850 4750
+Wire Wire Line
+	8850 5750 8850 5350
+Connection ~ 8850 4750
+Wire Wire Line
+	8850 4750 8850 5050
+Wire Notes Line
+	8800 5450 8900 5450
+Wire Notes Line
+	8900 5450 8900 5700
+Wire Notes Line
+	8900 5700 8800 5700
+Wire Notes Line
+	8800 5450 8800 5700
+Text Notes 8750 5900 1    39   ~ 0
 50ohm Microstrip
+$Comp
+L power:+6V #PWR?
+U 1 1 5BFE3C48
+P 4950 4950
+F 0 "#PWR?" H 4950 4800 50  0001 C CNN
+F 1 "+6V" V 4965 5123 50  0000 C CNN
+F 2 "" H 4950 4950 50  0001 C CNN
+F 3 "" H 4950 4950 50  0001 C CNN
+	1    4950 4950
+	-1   0    0    1
+$EndComp
+Wire Wire Line
+	5200 4950 4950 4950
+$Comp
+L power:+6V #PWR?
+U 1 1 5BFEFCC1
+P 3900 3950
+F 0 "#PWR?" H 3900 3800 50  0001 C CNN
+F 1 "+6V" V 3915 4123 50  0000 C CNN
+F 2 "" H 3900 3950 50  0001 C CNN
+F 3 "" H 3900 3950 50  0001 C CNN
+	1    3900 3950
+	1    0    0    -1
+$EndComp
+$Comp
+L Regulator_Linear:L7806 U2
+U 1 1 5BF5D575
+P 4850 2000
+F 0 "U2" H 4850 2242 50  0000 C CNN
+F 1 "L7806" H 4850 2151 50  0000 C CNN
+F 2 "My_Footprints:L7806ABV" H 4875 1850 50  0001 L CIN
+F 3 "http://www.st.com/content/ccc/resource/technical/document/datasheet/41/4f/b3/b0/12/d4/47/88/CD00000444.pdf/files/CD00000444.pdf/jcr:content/translations/en.CD00000444.pdf" H 4850 1950 50  0001 C CNN
+	1    4850 2000
+	1    0    0    -1
+$EndComp
+$Comp
+L power:+6V #PWR?
+U 1 1 5BFF778A
+P 5250 2000
+F 0 "#PWR?" H 5250 1850 50  0001 C CNN
+F 1 "+6V" V 5265 2173 50  0000 C CNN
+F 2 "" H 5250 2000 50  0001 C CNN
+F 3 "" H 5250 2000 50  0001 C CNN
+	1    5250 2000
+	1    0    0    -1
+$EndComp
 $EndSCHEMATC

Commit message: Finished Layout
Connections:
- net +6V: now also U1.13; no longer U1.10
- net at C1.1, R1.2, R2.1: now also U1.10, U1.9; no longer U1.1, U1.2
- net at U1.4, U1.5: now also U1.3; no longer U1.11
- net at U1.8: now also U1.1, U1.12; no longer U1.13
- new net: U1.11, U1.2
Other:
- moved on the sheet: U1A, U1C, U1D
Changed lines of the file:
@@
 L 74xx:74HC00 U1
 U 1 1 5BF5D5E6
-P 4800 4300
-F 0 "U1" H 4800 4625 50  0000 C CNN
-F 1 "74HC00" H 4800 4534 50  0000 C CNN
-F 2 "My_Footprints:HC00" H 4800 4300 50  0001 C CNN
-F 3 "http://www.ti.com/lit/gpn/sn74hc00" H 4800 4300 50  0001 C CNN
-	1    4800 4300
+P 6250 4450
+F 0 "U1" H 6250 4775 50  0000 C CNN
+F 1 "74HC00" H 6250 4684 50  0000 C CNN
+F 2 "My_Footprints:HC00" H 6250 4450 50  0001 C CNN
+F 3 "http://www.ti.com/lit/gpn/sn74hc00" H 6250 4450 50  0001 C CNN
+	1    6250 4450
 	1    0    0    -1
 $EndComp
@@
 L 74xx:74HC00 U1
 U 3 1 5BF5D77A
+P 4800 4300
+F 0 "U1" H 4800 4625 50  0000 C CNN
+F 1 "74HC00" H 4800 4534 50  0000 C CNN
+F 2 "My_Footprints:HC00" H 4800 4300 50  0001 C CNN
+F 3 "http://www.ti.com/lit/gpn/sn74hc00" H 4800 4300 50  0001 C CNN
+	3    4800 4300
+	1    0    0    -1
+$EndComp
+$Comp
+L 74xx:74HC00 U1
+U 4 1 5BF5D7E4
 P 5500 4850
 F 0 "U1" H 5500 5175 50  0000 C CNN
@@
 F 2 "My_Footprints:HC00" H 5500 4850 50  0001 C CNN
 F 3 "http://www.ti.com/lit/gpn/sn74hc00" H 5500 4850 50  0001 C CNN
-	3    5500 4850
-	1    0    0    -1
-$EndComp
-$Comp
-L 74xx:74HC00 U1
-U 4 1 5BF5D7E4
-P 6250 4450
-F 0 "U1" H 6250 4775 50  0000 C CNN
-F 1 "74HC00" H 6250 4684 50  0000 C CNN
-F 2 "My_Footprints:HC00" H 6250 4450 50  0001 C CNN
-F 3 "http://www.ti.com/lit/gpn/sn74hc00" H 6250 4450 50  0001 C CNN
-	4    6250 4450
+	4    5500 4850
 	1    0    0    -1
 $EndComp
@@
 50ohm Microstrip
 $Comp
-L power:+6V #PWR?
+L power:+6V #PWR0102
 U 1 1 5BFE3C48
 P 4950 4950
-F 0 "#PWR?" H 4950 4800 50  0001 C CNN
+F 0 "#PWR0102" H 4950 4800 50  0001 C CNN
 F 1 "+6V" V 4965 5123 50  0000 C CNN
 F 2 "" H 4950 4950 50  0001 C CNN
@@
 	5200 4950 4950 4950
 $Comp
-L power:+6V #PWR?
+L power:+6V #PWR0103
 U 1 1 5BFEFCC1
 P 3900 3950
-F 0 "#PWR?" H 3900 3800 50  0001 C CNN
+F 0 "#PWR0103" H 3900 3800 50  0001 C CNN
 F 1 "+6V" V 3915 4123 50  0000 C CNN
 F 2 "" H 3900 3950 50  0001 C CNN
@@
 $EndComp
 $Comp
-L power:+6V #PWR?
+L power:+6V #PWR0104
 U 1 1 5BFF778A
 P 5250 2000
-F 0 "#PWR?" H 5250 1850 50  0001 C CNN
+F 0 "#PWR0104" H 5250 1850 50  0001 C CNN
 F 1 "+6V" V 5265 2173 50  0000 C CNN
 F 2 "" H 5250 2000 50  0001 C CNN

Commit message: Nothing New
Parts:
- U1: footprint My_Footprints:HC00 -> digikey:SN74HC00DR
Changed lines of the file:
@@
 F 0 "U1" H 6250 4775 50  0000 C CNN
 F 1 "74HC00" H 6250 4684 50  0000 C CNN
-F 2 "My_Footprints:HC00" H 6250 4450 50  0001 C CNN
+F 2 "digikey:SN74HC00DR" H 6250 4450 50  0001 C CNN
 F 3 "http://www.ti.com/lit/gpn/sn74hc00" H 6250 4450 50  0001 C CNN
 	1    6250 4450
@@
 F 0 "U1" H 7100 4775 50  0000 C CNN
 F 1 "74HC00" H 7100 4684 50  0000 C CNN
-F 2 "My_Footprints:HC00" H 7100 4450 50  0001 C CNN
+F 2 "digikey:SN74HC00DR" H 7100 4450 50  0001 C CNN
 F 3 "http://www.ti.com/lit/gpn/sn74hc00" H 7100 4450 50  0001 C CNN
 	2    7100 4450
@@
 F 0 "U1" H 4800 4625 50  0000 C CNN
 F 1 "74HC00" H 4800 4534 50  0000 C CNN
-F 2 "My_Footprints:HC00" H 4800 4300 50  0001 C CNN
+F 2 "digikey:SN74HC00DR" H 4800 4300 50  0001 C CNN
 F 3 "http://www.ti.com/lit/gpn/sn74hc00" H 4800 4300 50  0001 C CNN
 	3    4800 4300
@@
 F 0 "U1" H 5500 5175 50  0000 C CNN
 F 1 "74HC00" H 5500 5084 50  0000 C CNN
-F 2 "My_Footprints:HC00" H 5500 4850 50  0001 C CNN
+F 2 "digikey:SN74HC00DR" H 5500 4850 50  0001 C CNN
 F 3 "http://www.ti.com/lit/gpn/sn74hc00" H 5500 4850 50  0001 C CNN
 	4    5500 4850
@@
 F 0 "U1" H 5880 3296 50  0000 L CNN
 F 1 "74HC00" H 5880 3205 50  0000 L CNN
-F 2 "My_Footprints:HC00" H 5650 3250 50  0001 C CNN
+F 2 "digikey:SN74HC00DR" H 5650 3250 50  0001 C CNN
 F 3 "http://www.ti.com/lit/gpn/sn74hc00" H 5650 3250 50  0001 C CNN
 	5    5650 3250

Commit message: Changed Schematic
Put all three circuits in the same schematic and added coax connectors
Parts:
- added C? (x8): C=100nF, Capacitor_SMD:C_0805_2012Metric, symbol Device:C
- added D? (x2): 1N4001, Diode_THT:D_DO-41_SOD81_P10.16mm_Horizontal, symbol Diode:1N4001
- added D? (x2): LED, LED_THT:LED_D5.0mm, symbol Device:LED
- added J? (x4): Conn_01x02_Male, My_Footprints:header_2_pins, symbol Connector:Conn_01x02_Male
- added J? (x5): Test Line, Connector_Coaxial:SMA_Amphenol_132289_EdgeMount, symbol EE173_Lab4-rescue:Conn_Coaxial-My_Connector
- added J? (x2): OSC, Connector_Coaxial:SMA_Amphenol_132289_EdgeMount, symbol EE173_Lab4-rescue:Conn_Coaxial-My_Connector
- added J?: BNC-T, symbol My_Connector:BNC-T
- added JP? (x12): Jumper, My_Footprints:header_2_pins, symbol Device:Jumper
- added R? (x2): R=10kohms, Resistor_SMD:R_0805_2012Metric, symbol Device:R
- added R? (x2): R=10kohm, Resistor_SMD:R_0805_2012Metric, symbol Device:R
- added R? (x2): R=1kohms, Resistor_SMD:R_0805_2012Metric, symbol Device:R
- added R? (x2): R=330ohms, Resistor_SMD:R_0805_2012Metric, symbol Device:R
- added R? (x2): R=50ohms, Resistor_SMD:R_0805_2012Metric, symbol Device:R
- added R? (x2): R=25ohms, Resistor_SMD:R_0805_2012Metric, symbol Device:R
- added U? (x10): 74HC00, digikey:SN74HC00DR, symbol 74xx:74HC00
- added U? (x2): L7806, My_Footprints:L7806ABV, symbol Regulator_Linear:L7806
- C1, C2, C3, C4: value C -> C=100nF
- J3: footprint My_Footprints:Vertical_BNC_Connector -> Connector_Coaxial:SMA_Amphenol_132289_EdgeMount
- J4: footprint My_Footprints:BNC_Connector -> Connector_Coaxial:SMA_Amphenol_132289_EdgeMount
- R1: value R -> R=10kohm
- R2: value R -> R=10kohms
- R3: value R -> R=330ohms
- R5: value R -> R=50ohms
- R6: value R -> R=25ohms
- R7: value R -> R=1kohms
Connections:
- net +6V: now also C?.2, C?.2, C?.2, C?.2, R?.1, R?.1, R?.2, R?.2, U?.13, U?.13, U?.14 (VCC), U?.14 (VCC), U?.3 (OUT), U?.3 (OUT)
- net GND: now also C?.1, C?.1, C?.1, C?.1, C?.1, C?.1, D?.1 (K), D?.1 (K), J?.2 (Ext), J?.2 (Ext), J?.2 (Ext), J?.2 (Ext), J?.2 (Ext), J?.2 (Ext), J?.2 (Ext), J?.2 (Pin_2), J?.2 (Pin_2), J?.2 (Pin_2), J?.2 (Pin_2), J?.3 (EXT), JP?.1, JP?.1, JP?.1, JP?.1, R?.2, R?.2, U?.2 (GND), U?.2 (GND), U?.7 (GND), U?.7 (GND)
- new net: J?.1 (Pin_1), JP?.1 (x2)
- new net: C?.1, R?.1, R?.2, U?.10, U?.9 (x2)
- new net: C?.2, JP?.2, JP?.2 (x2)
- new net: J?.1 (In), JP?.2, JP?.2, R?.1, R?.1, R?.1 (x2)
- new net: J?.1 (In), R?.2 (x2)
- new net: U?.1, U?.12, U?.8 (x2)
- new net: U?.11, U?.2 (x2)
- new net: U?.3, U?.4, U?.5 (x2)
- new net: JP?.1, JP?.1, JP?.1, U?.6 (x2)
- new net: C?.2, D?.1 (K), U?.1 (IN) (x2)
- new net: D?.2 (A), J?.1 (Pin_1) (x2)
- new net: D?.2 (A), R?.1 (x2)
- new net: JP?.2, R?.2 (x4)
- new net: J?.1 (IN1), J?.1 (In)
- new net: J?.1 (In), J?.2 (IN2)
- new net: J?.1 (In), J?.4 (IN1)
Other:
- note added: "-The TEST LINE on Luis’s Circuit will be connected to a t-type BNC connector.\n-Coaxial Cable will be connected either part of said t-type BNC Connector\n-The two lines of coaxial cable will be connected to Summer’s TEST LINE and Conner’s TEST LINE.\n"
- note added: "25ohm Microstrip"
- note added: "Conner’s Circuit:\n- 50ohm Microstrip\n-One Half of the Load Termination\n-DC Power Source and Signal Generator is not connected"
- note added: "Luis’s Circuit:\n-25ohm Microstrip (8inches)\n-Source End of the Bifurcated Line"
- note added: "Summer’s Circuit:\n- 50ohm Microstrip\n-One Half of the Load Termination\n-DC Power Source and Signal Generator is not connected"
- moved on the sheet: C1, C2, C3, C4, D1, D2, J1, J2, J3, J4, JP1, JP2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
